File: Maelstrom Boards/Acoustics/acoustics.sch (EAGLE design)
At the start: 175 parts

Commit message: Changed values
Parts:
- H4RF_C_O7, H4RF_C_O9, PA_C13, PF_C13: value 0.1uf -> 100nf
- PA_C3, PF_C3, SA_C3, SF_C3: value 10mF -> 10uF
Changed lines of the file:
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@@
 <part name="AGND46" library="supply1" library_urn="urn:adsk.eagle:library:371" deviceset="AGND" device=""/>
 <part name="PF_C4" library="resistor" library_urn="urn:adsk.eagle:library:348" deviceset="C-EU" device="C0603" package3d_urn="urn:adsk.eagle:package:26138/1" value="100nF"/>
-<part name="PF_C3" library="resistor" library_urn="urn:adsk.eagle:library:348" deviceset="C-EU" device="C0603" package3d_urn="urn:adsk.eagle:package:26138/1" value="10mF"/>
+<part name="PF_C3" library="resistor" library_urn="urn:adsk.eagle:library:348" deviceset="C-EU" device="C0603" package3d_urn="urn:adsk.eagle:package:26138/1" value="10uF"/>
 <part name="PF_C1" library="resistor" library_urn="urn:adsk.eagle:library:348" deviceset="C-EU" device="C0603" package3d_urn="urn:adsk.eagle:package:26138/1" value="1pF"/>
 <part name="PF_R2" library="resistor" library_urn="urn:adsk.eagle:library:348" deviceset="R-US_" device="R0603" package3d_urn="urn:adsk.eagle:package:26057/1" value="1 M"/>
@@
 <part name="AGND50" library="supply1" library_urn="urn:adsk.eagle:library:371" deviceset="AGND" device=""/>
 <part name="PA_C4" library="resistor" library_urn="urn:adsk.eagle:library:348" deviceset="C-EU" device="C0603" package3d_urn="urn:adsk.eagle:package:26138/1" value="100nF"/>
-<part name="PA_C3" library="resistor" library_urn="urn:adsk.eagle:library:348" deviceset="C-EU" device="C0603" package3d_urn="urn:adsk.eagle:package:26138/1" value="10mF"/>
+<part name="PA_C3" library="resistor" library_urn="urn:adsk.eagle:library:348" deviceset="C-EU" device="C0603" package3d_urn="urn:adsk.eagle:package:26138/1" value="10uF"/>
 <part name="PA_C1" library="resistor" library_urn="urn:adsk.eagle:library:348" deviceset="C-EU" device="C0603" package3d_urn="urn:adsk.eagle:package:26138/1" value="1pF"/>
 <part name="PA_R2" library="resistor" library_urn="urn:adsk.eagle:library:348" deviceset="R-US_" device="R0603" package3d_urn="urn:adsk.eagle:package:26057/1" value="1 M"/>
@@
 <part name="AGND54" library="supply1" library_urn="urn:adsk.eagle:library:371" deviceset="AGND" device=""/>
 <part name="SF_C4" library="resistor" library_urn="urn:adsk.eagle:library:348" deviceset="C-EU" device="C0603" package3d_urn="urn:adsk.eagle:package:26138/1" value="100nF"/>
-<part name="SF_C3" library="resistor" library_urn="urn:adsk.eagle:library:348" deviceset="C-EU" device="C0603" package3d_urn="urn:adsk.eagle:package:26138/1" value="10mF"/>
+<part name="SF_C3" library="resistor" library_urn="urn:adsk.eagle:library:348" deviceset="C-EU" device="C0603" package3d_urn="urn:adsk.eagle:package:26138/1" value="10uF"/>
 <part name="SF_C1" library="resistor" library_urn="urn:adsk.eagle:library:348" deviceset="C-EU" device="C0603" package3d_urn="urn:adsk.eagle:package:26138/1" value="1pF"/>
 <part name="SF_R2" library="resistor" library_urn="urn:adsk.eagle:library:348" deviceset="R-US_" device="R0603" package3d_urn="urn:adsk.eagle:package:26057/1" value="1 M"/>
@@
 <part name="AGND58" library="supply1" library_urn="urn:adsk.eagle:library:371" deviceset="AGND" device=""/>
 <part name="SA_C4" library="resistor" library_urn="urn:adsk.eagle:library:348" deviceset="C-EU" device="C0603" package3d_urn="urn:adsk.eagle:package:26138/1" value="100nF"/>
-<part name="SA_C3" library="resistor" library_urn="urn:adsk.eagle:library:348" deviceset="C-EU" device="C0603" package3d_urn="urn:adsk.eagle:package:26138/1" value="10mF"/>
+<part name="SA_C3" library="resistor" library_urn="urn:adsk.eagle:library:348" deviceset="C-EU" device="C0603" package3d_urn="urn:adsk.eagle:package:26138/1" value="10uF"/>
 <part name="SA_C1" library="resistor" library_urn="urn:adsk.eagle:library:348" deviceset="C-EU" device="C0603" package3d_urn="urn:adsk.eagle:package:26138/1" value="1pF"/>
 <part name="SA_R2" library="resistor" library_urn="urn:adsk.eagle:library:348" deviceset="R-US_" device="R0603" package3d_urn="urn:adsk.eagle:package:26057/1" value="1 M"/>
@@
 <part name="PF_R15" library="resistor" library_urn="urn:adsk.eagle:library:348" deviceset="R-US_" device="R0603" package3d_urn="urn:adsk.eagle:package:26057/1" value="121k"/>
 <part name="PF_C10" library="rcl" library_urn="urn:adsk.eagle:library:334" deviceset="C-EU" device="C0603" package3d_urn="urn:adsk.eagle:package:23616/2" value="10uf"/>
-<part name="PF_C13" library="rcl" library_urn="urn:adsk.eagle:library:334" deviceset="C-EU" device="C0603" package3d_urn="urn:adsk.eagle:package:23616/2" value="0.1uf"/>
+<part name="PF_C13" library="rcl" library_urn="urn:adsk.eagle:library:334" deviceset="C-EU" device="C0603" package3d_urn="urn:adsk.eagle:package:23616/2" value="100nf"/>
 <part name="PF_R16" library="resistor" library_urn="urn:adsk.eagle:library:348" deviceset="R-US_" device="R0603" package3d_urn="urn:adsk.eagle:package:26057/1" value="47m"/>
 <part name="PF_C12" library="rcl" library_urn="urn:adsk.eagle:library:334" deviceset="C-EU" device="C0603" package3d_urn="urn:adsk.eagle:package:23616/2" value="47uf"/>
@@
 <part name="PA_R15" library="resistor" library_urn="urn:adsk.eagle:library:348" deviceset="R-US_" device="R0603" package3d_urn="urn:adsk.eagle:package:26057/1" value="121k"/>
 <part name="PA_C10" library="rcl" library_urn="urn:adsk.eagle:library:334" deviceset="C-EU" device="C0603" package3d_urn="urn:adsk.eagle:package:23616/2" value="10uf"/>
-<part name="PA_C13" library="rcl" library_urn="urn:adsk.eagle:library:334" deviceset="C-EU" device="C0603" package3d_urn="urn:adsk.eagle:package:23616/2" value="0.1uf"/>
+<part name="PA_C13" library="rcl" library_urn="urn:adsk.eagle:library:334" deviceset="C-EU" device="C0603" package3d_urn="urn:adsk.eagle:package:23616/2" value="100nf"/>
 <part name="PA_R16" library="resistor" library_urn="urn:adsk.eagle:library:348" deviceset="R-US_" device="R0603" package3d_urn="urn:adsk.eagle:package:26057/1" value="47m"/>
 <part name="PA_C12" library="rcl" library_urn="urn:adsk.eagle:library:334" deviceset="C-EU" device="C0603" package3d_urn="urn:adsk.eagle:package:23616/2" value="47uf"/>
@@
 <part name="H4RF_R_6" library="resistor" library_urn="urn:adsk.eagle:library:348" deviceset="R-US_" device="R0603" package3d_urn="urn:adsk.eagle:package:26057/1" value="121k"/>
 <part name="H4RF_C_IN3" library="rcl" library_urn="urn:adsk.eagle:library:334" deviceset="C-EU" device="C0603" package3d_urn="urn:adsk.eagle:package:23616/2" value="10uf"/>
-<part name="H4RF_C_O7" library="rcl" library_urn="urn:adsk.eagle:library:334" deviceset="C-EU" device="C0603" package3d_urn="urn:adsk.eagle:package:23616/2" value="0.1uf"/>
+<part name="H4RF_C_O7" library="rcl" library_urn="urn:adsk.eagle:library:334" deviceset="C-EU" device="C0603" package3d_urn="urn:adsk.eagle:package:23616/2" value="100nf"/>
 <part name="H4RF_R_7" library="resistor" library_urn="urn:adsk.eagle:library:348" deviceset="R-US_" device="R0603" package3d_urn="urn:adsk.eagle:package:26057/1" value="47m"/>
 <part name="H4RF_C_O8" library="rcl" library_urn="urn:adsk.eagle:library:334" deviceset="C-EU" device="C0603" package3d_urn="urn:adsk.eagle:package:23616/2" value="47uf"/>
@@
 <part name="H4RF_R_8" library="resistor" library_urn="urn:adsk.eagle:library:348" deviceset="R-US_" device="R0603" package3d_urn="urn:adsk.eagle:package:26057/1" value="121k"/>
 <part name="H4RF_C_IN4" library="rcl" library_urn="urn:adsk.eagle:library:334" deviceset="C-EU" device="C0603" package3d_urn="urn:adsk.eagle:package:23616/2" value="10uf"/>
-<part name="H4RF_C_O9" library="rcl" library_urn="urn:adsk.eagle:library:334" deviceset="C-EU" device="C0603" package3d_urn="urn:adsk.eagle:package:23616/2" value="0.1uf"/>
+<part name="H4RF_C_O9" library="rcl" library_urn="urn:adsk.eagle:library:334" deviceset="C-EU" device="C0603" package3d_urn="urn:adsk.eagle:package:23616/2" value="100nf"/>
 <part name="H4RF_R_9" library="resistor" library_urn="urn:adsk.eagle:library:348" deviceset="R-US_" device="R0603" package3d_urn="urn:adsk.eagle:package:26057/1" value="47m"/>
 <part name="H4RF_C_O10" library="rcl" library_urn="urn:adsk.eagle:library:334" deviceset="C-EU" device="C0603" package3d_urn="urn:adsk.eagle:package:23616/2" value="47uf"/>

Commit message: New schematic template and converter fixes
Parts:
- removed ADC_H7, ADC_H8: ADS124S08IPBSRPBS0032A_L, ADS127L01_ADC:ADS124S08IPBSRPBS0032A_L
- removed H4ADC_C3, H4ADC_C4: 1uf, rcl:C-EUC0603K
- removed H4RF_C_3, H4RF_C_5, H4_C12, H4_C13, H4_C14, H4_C15, H4_C16, H4_C17, H4_C18, H4_C19, H4_C_POW3, H4_C_POW4: 1uf, rcl:C-EUC0603
- removed H4RF_C_IN3, H4RF_C_IN4: 10uf, rcl:C-EUC0603
- removed H4RF_C_O10, H4RF_C_O8: 47uf, rcl:C-EUC0603
- removed H4RF_C_O7, H4RF_C_O9: 100nf, rcl:C-EUC0603
- removed H4RF_R_6, H4RF_R_8: 121k, resistor:R-US_R0603
- removed H4RF_R_7, H4RF_R_9: 47m, resistor:R-US_R0603
- removed H4_R10, H4_R8: 10K, rcl:R-US_R0603
- removed H4_R5, H4_R9: 60.4k, rcl:R-US_R0603
- removed H4_REFGEN3, H4_REFGEN4: REF6025, REF6025:REF6025
- removed PF_C24, PF_C25, PF_C29, PF_C30: 270pF, resistor:C-EUC0603
- removed PF_C26, PF_C31: 1nF, resistor:C-EUC0603
- removed PF_C27, PF_C32: 470 pF, resistor:C-EUC0603
- removed PF_C28, PF_C33: 22nF, resistor:C-EUC0603
- removed PF_DA2, PF_DA3: THS4551, THS4551:THS4551
- removed PF_R29, PF_R32, PF_R39, PF_R42: 330, resistor:R-US_R0603
- removed PF_R30, PF_R40: 1.2K, resistor:R-US_R0603
- removed PF_R31, PF_R35, PF_R36, PF_R41, PF_R45, PF_R46: 1.2k, resistor:R-US_R0603
- removed PF_R33, PF_R34, PF_R43, PF_R44: 5, resistor:R-US_R0603
- removed PF_R37, PF_R38, PF_R47, PF_R48: 10, resistor:R-US_R0603
- removed U$1: 1X3, headers(2mm):1X3
- removed U$2: 2X8, headers(2mm):2X8
- added ADC_SA, ADC_SF: ADS124S08IPBSRPBS0032A_L, ADS127L01_ADC:ADS124S08IPBSRPBS0032A_L
- added FPGA_CON1: 2X8, headers(2mm):2X8
- added FPGA_CON2: 1X3, headers(2mm):1X3
- added SA_C10, SF_C10: 10uf, rcl:C-EUC0603
- added SA_C11, SA_C14, SA_C15, SA_C17, SA_C18, SA_C19, SF_C11, SF_C14, SF_C15, SF_C17, SF_C18, SF_C19: 1uf, rcl:C-EUC0603
- added SA_C12, SF_C12: 47uf, rcl:C-EUC0603
- added SA_C13, SF_C13: 100nf, rcl:C-EUC0603
- added SA_C16, SF_C16: 1uf, rcl:C-EUC0603K
- added SA_C5, SA_C9, SF_C5, SF_C9: 270pF, resistor:C-EUC0603
- added SA_C6, SF_C6: 470 pF, resistor:C-EUC0603
- added SA_C7, SF_C7: 1nF, resistor:C-EUC0603
- added SA_C8, SF_C8: 22nF, resistor:C-EUC0603
- added SA_DA, SF_DA: THS4551, THS4551:THS4551
- added SA_R10, SA_R14, SA_R5, SF_R10, SF_R14, SF_R5: 1.2k, resistor:R-US_R0603
- added SA_R11, SA_R7, SF_R11, SF_R7: 330, resistor:R-US_R0603
- added SA_R12, SA_R8, SF_R12, SF_R8: 5, resistor:R-US_R0603
- added SA_R13, SA_R9, SF_R13, SF_R9: 10, resistor:R-US_R0603
- added SA_R15, SF_R15: 121k, resistor:R-US_R0603
- added SA_R16, SF_R16: 47m, resistor:R-US_R0603
- added SA_R17, SF_R17: 60.4k, rcl:R-US_R0603
- added SA_R18, SF_R18: 10K, rcl:R-US_R0603
- added SA_R6, SF_R6: 1.2K, resistor:R-US_R0603
- added SA_REFGEN, SF_REFGEN: REF6025, REF6025:REF6025
Connections:
- net +3V3: now also ADC_SA.AVDD, ADC_SA.AVDD1, ADC_SA.DVDD, ADC_SA.HR, ADC_SA.RESET, ADC_SF.AVDD, ADC_SF.AVDD1, ADC_SF.DVDD, ADC_SF.HR, ADC_SF.RESET, FPGA_CON2.1, SA_C10.2, SA_C16.1, SA_C19.1, SA_DA.VS+, SA_REFGEN.EN, SA_REFGEN.VIN, SF_C10.2, SF_C16.1, SF_C19.1, SF_DA.VS+, SF_REFGEN.EN, SF_REFGEN.VIN; no longer ADC_H7.AVDD, ADC_H7.AVDD1, ADC_H7.DVDD, ADC_H7.HR, ADC_H7.RESET, ADC_H8.AVDD, ADC_H8.AVDD1, ADC_H8.DVDD, ADC_H8.HR, ADC_H8.RESET, H4ADC_C3.1, H4ADC_C4.1, H4RF_C_IN3.2, H4RF_C_IN4.2, H4_C_POW3.1, H4_C_POW4.1, H4_REFGEN3.EN, H4_REFGEN3.VIN, H4_REFGEN4.EN, H4_REFGEN4.VIN, PF_DA2.VS+, PF_DA3.VS+, U$1.1
- net +5V: now also FPGA_CON2.2; no longer U$1.2
- net AMPED_SA: now also SA_R6.1; no longer PF_R40.1
- net AMPED_SF: now also SF_R6.1; no longer PF_R30.1
- net CLK: now also ADC_SA.CLK, ADC_SF.CLK, FPGA_CON1.10; no longer ADC_H7.CLK, ADC_H8.CLK, U$2.10
- net DIFF_N_SA: now also ADC_SA.AINN, SA_C8.1, SA_R9.2; no longer ADC_H8.AINN, PF_C33.1, PF_R47.2
- net DIFF_N_SF: now also ADC_SF.AINN, SF_C8.1, SF_R9.2; no longer ADC_H7.AINN, PF_C28.1, PF_R37.2
- net DIFF_P_SA: now also ADC_SA.AINP, SA_C8.2, SA_R13.2; no longer ADC_H8.AINP, PF_C33.2, PF_R48.2
- net DIFF_P_SF: now also ADC_SF.AINP, SF_C8.2, SF_R13.2; no longer ADC_H7.AINP, PF_C28.2, PF_R38.2
- net DOUT_PA: now also FPGA_CON1.4; no longer U$2.4
- net DOUT_PF: now also FPGA_CON1.2; no longer U$2.2
- net DOUT_SA: now also ADC_SA.DOUT, FPGA_CON1.8; no longer ADC_H8.DOUT, U$2.8
- net DOUT_SF: now also ADC_SF.DOUT, FPGA_CON1.6; no longer ADC_H7.DOUT, U$2.6
- net DRDY_PA: now also FPGA_CON1.3; no longer U$2.3
- net DRDY_PF: now also FPGA_CON1.1; no longer U$2.1
- net DRDY_SA: now also ADC_SA.DRDY, FPGA_CON1.7; no longer ADC_H8.DRDY, U$2.7
- net DRDY_SF: now also ADC_SF.DRDY, FPGA_CON1.5; no longer ADC_H7.DRDY, U$2.5
- net GND: now also ADC_SA.AGND, ADC_SA.AGND1, ADC_SA.CS, ADC_SA.DAISYIN, ADC_SA.DGND, ADC_SA.DIN, ADC_SA.FILTER0, ADC_SA.FILTER1, ADC_SA.FORMAT, ADC_SA.FSMODE, ADC_SA.OSR0, ADC_SA.OSR1, ADC_SA.REFN, ADC_SF.AGND, ADC_SF.AGND1, ADC_SF.CS, ADC_SF.DAISYIN, ADC_SF.DGND, ADC_SF.DIN, ADC_SF.FILTER0, ADC_SF.FILTER1, ADC_SF.FORMAT, ADC_SF.FSMODE, ADC_SF.OSR0, ADC_SF.OSR1, ADC_SF.REFN, FPGA_CON1.15, FPGA_CON1.16, FPGA_CON2.3, SA_C10.1, SA_C11.1, SA_C13.1, SA_C14.1, SA_C15.1, SA_C16.2, SA_C17.2, SA_C18.1, SA_C19.2, SA_DA.VS-, SA_R10.1, SA_R15.1, SA_R16.1, SA_R17.2, SA_R18.2, SA_REFGEN.GND_F, SA_REFGEN.GND_S, SF_C10.1, SF_C11.1, SF_C13.1, SF_C14.1, SF_C15.1, SF_C16.2, SF_C17.2, SF_C18.1, SF_C19.2, SF_DA.VS-, SF_R10.1, SF_R15.1, SF_R16.1, SF_R17.2, SF_R18.2, SF_REFGEN.GND_F, SF_REFGEN.GND_S; no longer ADC_H7.AGND, ADC_H7.AGND1, ADC_H7.CS, ADC_H7.DAISYIN, ADC_H7.DGND, ADC_H7.DIN, ADC_H7.FILTER0, ADC_H7.FILTER1, ADC_H7.FORMAT, ADC_H7.FSMODE, ADC_H7.OSR0, ADC_H7.OSR1, ADC_H7.REFN, ADC_H8.AGND, ADC_H8.AGND1, ADC_H8.CS, ADC_H8.DAISYIN, ADC_H8.DGND, ADC_H8.DIN, ADC_H8.FILTER0, ADC_H8.FILTER1, ADC_H8.FORMAT, ADC_H8.FSMODE, ADC_H8.OSR0, ADC_H8.OSR1, ADC_H8.REFN, H4ADC_C3.2, H4ADC_C4.2, H4RF_C_3.1, H4RF_C_5.1, H4RF_C_IN3.1, H4RF_C_IN4.1, H4RF_C_O7.1, H4RF_C_O9.1, H4RF_R_6.1, H4RF_R_7.1, H4RF_R_8.1, H4RF_R_9.1, H4_C12.1, H4_C13.1, H4_C14.2, H4_C15.1, H4_C16.1, H4_C17.1, H4_C18.2, H4_C19.1, H4_C_POW3.2, H4_C_POW4.2, H4_R10.2, H4_R5.2, H4_R8.2, H4_R9.2, H4_REFGEN3.GND_F, H4_REFGEN3.GND_S, H4_REFGEN4.GND_F, H4_REFGEN4.GND_S, PF_DA2.VS-, PF_DA3.VS-, PF_R31.1, PF_R41.1, U$1.3, U$2.15, U$2.16
- net N$10: now also SF_C5.1, SF_C7.1, SF_DA.IN+, SF_R7.2; no longer PF_C24.1, PF_C26.1, PF_DA2.IN+, PF_R29.2
- net N$11: now also SF_C7.2, SF_C9.1, SF_DA.IN-, SF_R11.2; no longer PF_C25.1, PF_C26.2, PF_DA2.IN-, PF_R32.2
- net N$118: now also SF_C11.2, SF_REFGEN.FILT; no longer H4RF_C_3.2, H4_REFGEN3.FILT
- net N$12: now also SF_C6.1, SF_R5.1, SF_R6.2, SF_R7.1; no longer PF_C27.1, PF_R29.1, PF_R30.2, PF_R35.1
- net N$121: now also SF_R15.2, SF_REFGEN.SS; no longer H4RF_R_6.2, H4_REFGEN3.SS
- net N$124: now also SF_C12.1, SF_R16.2; no longer H4RF_C_O8.1, H4RF_R_7.2
- net N$129: now also SA_C11.2, SA_REFGEN.FILT; no longer H4RF_C_5.2, H4_REFGEN4.FILT
- net N$13: now also SF_C6.2, SF_R10.2, SF_R11.1, SF_R14.1; no longer PF_C27.2, PF_R31.2, PF_R32.1, PF_R36.1
- net N$130: now also SA_R15.2, SA_REFGEN.SS; no longer H4RF_R_8.2, H4_REFGEN4.SS
- net N$131: now also SA_C12.1, SA_R16.2; no longer H4RF_C_O10.1, H4RF_R_9.2
- net N$14: now also SF_C9.2, SF_DA.OUT+, SF_R12.1; no longer PF_C25.2, PF_DA2.OUT+, PF_R34.1
- net N$15: now also SF_R5.2, SF_R8.2, SF_R9.1; no longer PF_R33.2, PF_R35.2, PF_R37.1
- net N$156: now also ADC_SF.LVDD, SF_C15.2; no longer ADC_H7.LVDD, H4_C13.2
- net N$157: now also ADC_SF.INTLDO, SF_R18.1; no longer ADC_H7.INTLDO, H4_R8.1
- net N$158: now also ADC_SF.REXT, SF_R17.1; no longer ADC_H7.REXT, H4_R5.1
- net N$159: now also ADC_SF.CAP2, SF_C17.1; no longer ADC_H7.CAP2, H4_C14.1
- net N$16: now also SF_R12.2, SF_R13.1, SF_R14.2; no longer PF_R34.2, PF_R36.2, PF_R38.1
- net N$160: now also ADC_SF.CAP3, SF_C18.2; no longer ADC_H7.CAP3, H4_C15.2
- net N$161: now also ADC_SF.CAP1, SF_C14.2; no longer ADC_H7.CAP1, H4_C12.2
- net N$162: now also ADC_SA.LVDD, SA_C15.2; no longer ADC_H8.LVDD, H4_C17.2
- net N$163: now also ADC_SA.INTLDO, SA_R18.1; no longer ADC_H8.INTLDO, H4_R10.1
- net N$164: now also ADC_SA.REXT, SA_R17.1; no longer ADC_H8.REXT, H4_R9.1
- net N$165: now also ADC_SA.CAP2, SA_C17.1; no longer ADC_H8.CAP2, H4_C18.1
- net N$166: now also ADC_SA.CAP3, SA_C18.2; no longer ADC_H8.CAP3, H4_C19.2
- net N$167: now also ADC_SA.CAP1, SA_C14.2; no longer ADC_H8.CAP1, H4_C16.2
- net N$17: now also SA_C5.2, SA_DA.OUT-, SA_R8.1; no longer PF_C29.2, PF_DA3.OUT-, PF_R43.1
- net N$18: now also SA_C5.1, SA_C7.1, SA_DA.IN+, SA_R7.2; no longer PF_C29.1, PF_C31.1, PF_DA3.IN+, PF_R39.2
- net N$19: now also SA_C7.2, SA_C9.1, SA_DA.IN-, SA_R11.2; no longer PF_C30.1, PF_C31.2, PF_DA3.IN-, PF_R42.2
- net N$20: now also SA_C6.1, SA_R5.1, SA_R6.2, SA_R7.1; no longer PF_C32.1, PF_R39.1, PF_R40.2, PF_R45.1
- net N$21: now also SA_C6.2, SA_R10.2, SA_R11.1, SA_R14.1; no longer PF_C32.2, PF_R41.2, PF_R42.1, PF_R46.1
- net N$22: now also SA_C9.2, SA_DA.OUT+, SA_R12.1; no longer PF_C30.2, PF_DA3.OUT+, PF_R44.1
- net N$23: now also SA_R5.2, SA_R8.2, SA_R9.1; no longer PF_R43.2, PF_R45.2, PF_R47.1
- net N$24: now also SA_R12.2, SA_R13.1, SA_R14.2; no longer PF_R44.2, PF_R46.2, PF_R48.1
- net N$9: now also SF_C5.2, SF_DA.OUT-, SF_R8.1; no longer PF_C24.2, PF_DA2.OUT-, PF_R33.1
- net REF_SA: now also ADC_SA.REFP, SA_C12.2, SA_C13.2, SA_REFGEN.OUT_F, SA_REFGEN.OUT_S; no longer ADC_H8.REFP, H4RF_C_O10.2, H4RF_C_O9.2, H4_REFGEN4.OUT_F, H4_REFGEN4.OUT_S
- net REF_SF: now also ADC_SF.REFP, SF_C12.2, SF_C13.2, SF_REFGEN.OUT_F, SF_REFGEN.OUT_S; no longer ADC_H7.REFP, H4RF_C_O7.2, H4RF_C_O8.2, H4_REFGEN3.OUT_F, H4_REFGEN3.OUT_S
- net SCLK: now also ADC_SA.SCLK, ADC_SF.SCLK, FPGA_CON1.9; no longer ADC_H7.SCLK, ADC_H8.SCLK, U$2.9
- net START: now also ADC_SA.START, ADC_SF.START, FPGA_CON1.12; no longer ADC_H7.START, ADC_H8.START, U$2.12
Other:
- note added: "Electrical Team"
- note added: "Underwater Robotics Team Ohio State University"
- moved on the sheet: ADC_PA, ADC_PF, C1, C2, C3, C4, C5, PA_C1, PA_C10, PA_C11, PA_C12, PA_C13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

Commit message: Touching up acoustics
Other:
- note added: "ADCs"
- note added: "Connectors & Caps"
- note added: "Differential Amps"
- note added: "Pre-amps"
- note added: "Reference Generators"
- note removed: "Electrical Team"
- moved on the sheet: ADC_PF, ADC_SF, PA_C1, PA_C10, PA_C11, PA_C12, PA_C13, PA_C2, PA_C3, PA_C4, PA_R1, PA_R15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
