File: Maelstrom Boards/Converter/Converter.sch (EAGLE design)
At the start: 1 part

Commit message: converter work
Parts:
- added 12VCONVERTER, 3.3VCONVERTER, 5VCONVERTER: CONVERTER, converter:CONVERTER
- added BALANCEDRAWIN: 39-30-06, con-molex-mini-fit:39-30-06
- added C1, C12, C7: (no value), rcl:CPOL-USE3.5-10
- added C10, C13, C14, C15, C3, C4, C5, C8, C9: (no value), resistor:C-USC1206K
- added C11, C2, C6: (no value), rcl:CPOL-USE5-13
- added DIAMOND: 43045-08, con-molex-micro-fit:43045-08
- added JETSON, PNUEMATICS: 39-30-02, con-molex-mini-fit:39-30-02
- added L1, L2, L3: (no value), rcl:L-USWE-TPC
- added Q1, Q2, Q3: BSS295, transistor-fet:BSS295
- added R4: 4.47 K, rcl:R-US_0207/10
- added R5: 1.41 K, rcl:R-US_0207/10
- added R6: 7.6 K, rcl:R-US_0207/10
Connections:
- new net +12V: 12VCONVERTER.7,SENSE+, 12VCONVERTER.8,VOUT(+)
- new net +3V3: 3.3VCONVERTER.7,SENSE+, 3.3VCONVERTER.8,VOUT(+), U$1.3.3V
- new net +5V: 5VCONVERTER.7,SENSE+, 5VCONVERTER.8,VOUT(+), U$1.5V
- new net 12VCURRENTOUT: C3.1, C4.1, C5.1, DIAMOND.1, DIAMOND.2, DIAMOND.3, DIAMOND.4, JETSON.1, PNUEMATICS.1
- new net 12VFILTERED+: 12VCONVERTER.1,VIN(+)
- new net 12VON: Q1.G, U$1.12V_ON/OFF
- new net 3.3VFILTERED+: 3.3VCONVERTER.1,VIN(+)
- new net 3.3VON: Q3.G, U$1.3.3V_ON/OFF
- new net 5VFILTERED+: 5VCONVERTER.1,VIN(+)
- new net 5VON: Q2.G, U$1.5V_ON_OFF
- new net AGND: 12VCONVERTER.3,VIN(-)/GND, 12VCONVERTER.4,VOUT(-)/GND, 3.3VCONVERTER.3,VIN(-)/GND, 3.3VCONVERTER.4,VOUT(-)/GND, 5VCONVERTER.3,VIN(-)/GND, 5VCONVERTER.4,VOUT(-)/GND, Q1.S, Q2.S, Q3.S, R4.1, R5.1, R6.1, U$1.GND
- new net BALANCED+: BALANCEDRAWIN.1, BALANCEDRAWIN.2, BALANCEDRAWIN.3, C1.+, C12.+, C7.+, L1.1, L2.1, L3.1
- new net BALANCED-: BALANCEDRAWIN.4, BALANCEDRAWIN.5, BALANCEDRAWIN.6, C1.-, C11.-, C12.-, C2.-, C6.-, C7.-
- new net CMGND: C3.2, C4.2, C5.2, DIAMOND.5, DIAMOND.6, DIAMOND.7, DIAMOND.8, JETSON.2, PNUEMATICS.2
- new net N$1: 5VCONVERTER.6,TRIM, R4.2
- new net N$10: C13.1, C14.1, C15.1
- new net N$11: C13.2, C14.2, C15.2
- new net N$13: 12VCONVERTER.2,ON/OFF, Q1.D
- new net N$16: 5VCONVERTER.2,ON/OFF, Q2.D
- new net N$17: 3.3VCONVERTER.6,TRIM, R6.2
- new net N$19: 3.3VCONVERTER.2,ON/OFF, Q3.D
- new net N$2: 12VCONVERTER.6,TRIM, R5.2
- new net N$3: C2.+, L1.2
- new net N$5: C6.+, L2.2
- new net N$6: C10.1, C8.1, C9.1
- new net N$7: C10.2, C8.2, C9.2
- new net N$9: C11.+, L3.2

Commit message: Converter work
Parts:
- added R1: 10K, rcl:R-US_R0603
- added R2: 1.41 K, rcl:R-US_R0603
- added R3, R7, R8, R9: 4.47 K, rcl:R-US_R0603
- C1, C7: value (none) -> 1000 uF
- C10, C13, C14, C15, C3, C4, C5, C8, C9: value (none) -> 47 uF
- C11, C2, C6: value (none) -> 330 uF; device rcl:CPOL-USE5-13 -> rcl:CPOL-USE3.5-8
- C12: value (none) -> 1000
- L1, L2, L3: value (none) -> 1 uH
- R4, R5, R6: device rcl:R-US_0207/10 -> rcl:R-US_R0603
Connections:
- net N$1 renamed 5VTRIM
- net N$10 renamed +3.3V
- net N$13 renamed 12VON-CON
- net N$16 renamed 5VON-CON
- net N$17 renamed 3.3VTRIM
- net N$19 renamed 3.3VON-CON
- net N$2 renamed 12VTRIM
- removed net 12VCURRENTOUT: C3.1, C4.1, C5.1, DIAMOND.1, DIAMOND.2, DIAMOND.3, DIAMOND.4, JETSON.1, PNUEMATICS.1
- removed net CMGND: C3.2, C4.2, C5.2, DIAMOND.5, DIAMOND.6, DIAMOND.7, DIAMOND.8, JETSON.2, PNUEMATICS.2
- removed net N$11: C13.2, C14.2, C15.2
- removed net N$3: C2.+, L1.2
- removed net N$5: C6.+, L2.2
- removed net N$6: C10.1, C8.1, C9.1
- removed net N$7: C10.2, C8.2, C9.2
- removed net N$9: C11.+, L3.2
- net +12V: now also C3.1, C4.1, C5.1, DIAMOND.1, DIAMOND.2, DIAMOND.3, DIAMOND.4, JETSON.1, PNUEMATICS.1
- net +5V: now also C10.1, C8.1, C9.1
- net 12VFILTERED+: now also C2.+, L1.2
- net 12VON: now also R1.1, R2.2
- net 3.3VFILTERED+: now also C11.+, L3.2
- net 3.3VON: now also R8.1, R9.2
- net 5VFILTERED+: now also C6.+, L2.2
- net 5VON: now also R3.1, R7.2
- net AGND: now also C10.2, C13.2, C14.2, C15.2, C3.2, C4.2, C5.2, C8.2, C9.2, DIAMOND.5, DIAMOND.6, DIAMOND.7, DIAMOND.8, JETSON.2, PNUEMATICS.2, R2.1, R7.1, R9.1
- net BALANCED+: now also R1.2, R3.2, R8.2
Other:
- moved on the sheet: C11, C2, Q1

Commit message: Converter board
Parts:
- R2: value 1.41 K -> 1.35K
- R3, R8: value 4.47 K -> 10K
- R7, R9: value 4.47 K -> 1.35K
Connections:
- removed net BALANCED-: BALANCEDRAWIN.4, BALANCEDRAWIN.5, BALANCEDRAWIN.6, C1.-, C11.-, C12.-, C2.-, C6.-, C7.-
- net AGND: now also BALANCEDRAWIN.4, BALANCEDRAWIN.5, BALANCEDRAWIN.6, C1.-, C11.-, C12.-, C2.-, C6.-, C7.-
Changed lines of the file:
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@@
 <part name="P+4" library="supply1" library_urn="urn:adsk.eagle:library:371" deviceset="V+" device=""/>
 <part name="R1" library="rcl" library_urn="urn:adsk.eagle:library:334" deviceset="R-US_" device="R0603" package3d_urn="urn:adsk.eagle:package:23555/2" value="10K"/>
-<part name="R2" library="rcl" library_urn="urn:adsk.eagle:library:334" deviceset="R-US_" device="R0603" package3d_urn="urn:adsk.eagle:package:23555/2" value="1.41 K"/>
+<part name="R2" library="rcl" library_urn="urn:adsk.eagle:library:334" deviceset="R-US_" device="R0603" package3d_urn="urn:adsk.eagle:package:23555/2" value="1.35K"/>
 <part name="P+5" library="supply1" library_urn="urn:adsk.eagle:library:371" deviceset="V+" device=""/>
-<part name="R3" library="rcl" library_urn="urn:adsk.eagle:library:334" deviceset="R-US_" device="R0603" package3d_urn="urn:adsk.eagle:package:23555/2" value="4.47 K"/>
-<part name="R7" library="rcl" library_urn="urn:adsk.eagle:library:334" deviceset="R-US_" device="R0603" package3d_urn="urn:adsk.eagle:package:23555/2" value="4.47 K"/>
+<part name="R3" library="rcl" library_urn="urn:adsk.eagle:library:334" deviceset="R-US_" device="R0603" package3d_urn="urn:adsk.eagle:package:23555/2" value="10K"/>
+<part name="R7" library="rcl" library_urn="urn:adsk.eagle:library:334" deviceset="R-US_" device="R0603" package3d_urn="urn:adsk.eagle:package:23555/2" value="1.35K"/>
 <part name="P+6" library="supply1" library_urn="urn:adsk.eagle:library:371" deviceset="V+" device=""/>
-<part name="R8" library="rcl" library_urn="urn:adsk.eagle:library:334" deviceset="R-US_" device="R0603" package3d_urn="urn:adsk.eagle:package:23555/2" value="4.47 K"/>
-<part name="R9" library="rcl" library_urn="urn:adsk.eagle:library:334" deviceset="R-US_" device="R0603" package3d_urn="urn:adsk.eagle:package:23555/2" value="4.47 K"/>
+<part name="R8" library="rcl" library_urn="urn:adsk.eagle:library:334" deviceset="R-US_" device="R0603" package3d_urn="urn:adsk.eagle:package:23555/2" value="10K"/>
+<part name="R9" library="rcl" library_urn="urn:adsk.eagle:library:334" deviceset="R-US_" device="R0603" package3d_urn="urn:adsk.eagle:package:23555/2" value="1.35K"/>
 <part name="P+7" library="supply1" library_urn="urn:adsk.eagle:library:371" deviceset="V+" device=""/>
+<part name="AGND8" library="supply1" library_urn="urn:adsk.eagle:library:371" deviceset="AGND" device=""/>
 </parts>
 <sheets>
@@
 <instance part="C11" gate="G$1" x="40.64" y="106.68"/>
 <instance part="P+4" gate="1" x="8.89" y="271.78"/>
+<instance part="AGND8" gate="VR1" x="-29.21" y="231.14"/>
 </instances>
 <busses>
 </busses>
 <nets>
-<net name="BALANCED-" class="0">
-<segment>
-<pinref part="BALANCEDRAWIN" gate="G$1" pin="4"/>
-<wire x1="-16.51" y1="256.54" x2="-16.51" y2="254" width="0.1524" layer="91"/>
-<pinref part="BALANCEDRAWIN" gate="G$1" pin="6"/>
-<junction x="-16.51" y="254"/>
-<wire x1="-16.51" y1="254" x2="-16.51" y2="246.38" width="0.1524" layer="91"/>
-<wire x1="-31.75" y1="246.38" x2="-21.59" y2="246.38" width="0.1524" layer="91"/>
-<pinref part="BALANCEDRAWIN" gate="G$1" pin="5"/>
-<wire x1="-21.59" y1="246.38" x2="-16.51" y2="246.38" width="0.1524" layer="91"/>
-<wire x1="-31.75" y1="254" x2="-31.75" y2="246.38" width="0.1524" layer="91"/>
-<wire x1="40.64" y1="176.53" x2="8.89" y2="176.53" width="0.1524" layer="91"/>
-<wire x1="8.89" y1="176.53" x2="-21.59" y2="176.53" width="0.1524" layer="91"/>
-<wire x1="-21.59" y1="246.38" x2="-21.59" y2="176.53" width="0.1524" layer="91"/>
-<junction x="-21.59" y="246.38"/>
-<pinref part="C1" gate="G$1" pin="-"/>
-<wire x1="8.89" y1="176.53" x2="8.89" y2="180.594" width="0.1524" layer="91"/>
-<junction x="8.89" y="176.53"/>
-<pinref part="C7" gate="G$1" pin="-"/>
-<wire x1="40.64" y1="130.81" x2="10.16" y2="130.81" width="0.1524" layer="91"/>
-<wire x1="10.16" y1="130.81" x2="10.16" y2="134.874" width="0.1524" layer="91"/>
-<wire x1="-21.59" y1="176.53" x2="-21.59" y2="130.81" width="0.1524" layer="91"/>
-<wire x1="-21.59" y1="130.81" x2="10.16" y2="130.81" width="0.1524" layer="91"/>
-<junction x="-21.59" y="176.53"/>
-<junction x="10.16" y="130.81"/>
-<wire x1="40.64" y1="96.52" x2="10.16" y2="96.52" width="0.1524" layer="91"/>
-<pinref part="C12" gate="G$1" pin="-"/>
-<wire x1="10.16" y1="96.52" x2="10.16" y2="100.584" width="0.1524" layer="91"/>
-<wire x1="-21.59" y1="130.81" x2="-21.59" y2="96.52" width="0.1524" layer="91"/>
-<wire x1="-21.59" y1="96.52" x2="10.16" y2="96.52" width="0.1524" layer="91"/>
-<junction x="-21.59" y="130.81"/>
-<junction x="10.16" y="96.52"/>
-<pinref part="C6" gate="G$1" pin="-"/>
-<wire x1="40.64" y1="130.81" x2="40.64" y2="134.62" width="0.1524" layer="91"/>
-<pinref part="C11" gate="G$1" pin="-"/>
-<wire x1="40.64" y1="96.52" x2="40.64" y2="101.6" width="0.1524" layer="91"/>
-<pinref part="C2" gate="G$1" pin="-"/>
-<wire x1="40.64" y1="176.53" x2="40.64" y2="180.34" width="0.1524" layer="91"/>
-</segment>
-</net>
 <net name="+12V" class="0">
 <segment>
@@
 <junction x="160.02" y="96.52"/>
 <label x="167.64" y="93.98" size="1.778" layer="95"/>
+</segment>
+<segment>
+<pinref part="BALANCEDRAWIN" gate="G$1" pin="4"/>
+<wire x1="-16.51" y1="256.54" x2="-16.51" y2="254" width="0.1524" layer="91"/>
+<pinref part="BALANCEDRAWIN" gate="G$1" pin="6"/>
+<junction x="-16.51" y="254"/>
+<wire x1="-16.51" y1="254" x2="-16.51" y2="246.38" width="0.1524" layer="91"/>
+<wire x1="-31.75" y1="246.38" x2="-29.21" y2="246.38" width="0.1524" layer="91"/>
+<pinref part="BALANCEDRAWIN" gate="G$1" pin="5"/>
+<wire x1="-29.21" y1="246.38" x2="-21.59" y2="246.38" width="0.1524" layer="91"/>
+<wire x1="-21.59" y1="246.38" x2="-16.51" y2="246.38" width="0.1524" layer="91"/>
+<wire x1="-31.75" y1="254" x2="-31.75" y2="246.38" width="0.1524" layer="91"/>
+<wire x1="40.64" y1="176.53" x2="8.89" y2="176.53" width="0.1524" layer="91"/>
+<wire x1="8.89" y1="176.53" x2="-21.59" y2="176.53" width="0.1524" layer="91"/>
+<wire x1="-21.59" y1="246.38" x2="-21.59" y2="176.53" width="0.1524" layer="91"/>
+<junction x="-21.59" y="246.38"/>
+<pinref part="C1" gate="G$1" pin="-"/>
+<wire x1="8.89" y1="176.53" x2="8.89" y2="180.594" width="0.1524" layer="91"/>
+<junction x="8.89" y="176.53"/>
+<pinref part="C7" gate="G$1" pin="-"/>
+<wire x1="40.64" y1="130.81" x2="10.16" y2="130.81" width="0.1524" layer="91"/>
+<wire x1="10.16" y1="130.81" x2="10.16" y2="134.874" width="0.1524" layer="91"/>
+<wire x1="-21.59" y1="176.53" x2="-21.59" y2="130.81" width="0.1524" layer="91"/>
+<wire x1="-21.59" y1="130.81" x2="10.16" y2="130.81" width="0.1524" layer="91"/>
+<junction x="-21.59" y="176.53"/>
+<junction x="10.16" y="130.81"/>
+<wire x1="40.64" y1="96.52" x2="10.16" y2="96.52" width="0.1524" layer="91"/>
+<pinref part="C12" gate="G$1" pin="-"/>
+<wire x1="10.16" y1="96.52" x2="10.16" y2="100.584" width="0.1524" layer="91"/>
+<wire x1="-21.59" y1="130.81" x2="-21.59" y2="96.52" width="0.1524" layer="91"/>
+<wire x1="-21.59" y1="96.52" x2="10.16" y2="96.52" width="0.1524" layer="91"/>
+<junction x="-21.59" y="130.81"/>
+<junction x="10.16" y="96.52"/>
+<pinref part="C6" gate="G$1" pin="-"/>
+<wire x1="40.64" y1="130.81" x2="40.64" y2="134.62" width="0.1524" layer="91"/>
+<pinref part="C11" gate="G$1" pin="-"/>
+<wire x1="40.64" y1="96.52" x2="40.64" y2="101.6" width="0.1524" layer="91"/>
+<pinref part="C2" gate="G$1" pin="-"/>
+<wire x1="40.64" y1="176.53" x2="40.64" y2="180.34" width="0.1524" layer="91"/>
+<pinref part="AGND8" gate="VR1" pin="AGND"/>
+<wire x1="-29.21" y1="233.68" x2="-29.21" y2="246.38" width="0.1524" layer="91"/>
+<junction x="-29.21" y="246.38"/>
 </segment>
 </net>
@@
 <wire x1="-16.51" y1="40.64" x2="-19.05" y2="40.64" width="0.1524" layer="91"/>
 <junction x="-16.51" y="38.1"/>
-<pinref part="R7" gate="G$1" pin="1"/>
-<wire x1="-43.18" y1="27.94" x2="-26.67" y2="27.94" width="0.1524" layer="91"/>
 <wire x1="-26.67" y1="27.94" x2="-26.67" y2="35.56" width="0.1524" layer="91"/>
 <wire x1="-26.67" y1="35.56" x2="-16.51" y2="35.56" width="0.1524" layer="91"/>
 <junction x="-16.51" y="35.56"/>
+<pinref part="R7" gate="G$1" pin="1"/>
+<wire x1="-43.18" y1="27.94" x2="-26.67" y2="27.94" width="0.1524" layer="91"/>
 </segment>
 <segment>
@@
 <wire x1="-43.18" y1="43.18" x2="-43.18" y2="40.64" width="0.1524" layer="91"/>
 <wire x1="-43.18" y1="40.64" x2="-39.37" y2="40.64" width="0.1524" layer="91"/>
-<pinref part="R7" gate="G$1" pin="2"/>
-<wire x1="-43.18" y1="40.64" x2="-43.18" y2="38.1" width="0.1524" layer="91"/>
 <junction x="-43.18" y="40.64"/>
 <wire x1="-43.18" y1="40.64" x2="-50.8" y2="40.64" width="0.1524" layer="91"/>
-</segment>
-</net>
+<pinref part="R7" gate="G$1" pin="2"/>
+<wire x1="-43.18" y1="38.1" x2="-43.18" y2="40.64" width="0.1524" layer="91"/>
+</segment>
+</net>

Commit message: Converter layout finished
Connections:
- removed net +3.3V: C13.1, C14.1, C15.1
- net +3V3: now also C13.1, C14.1, C15.1
Changed lines of the file:
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@@
 <part name="P+7" library="supply1" library_urn="urn:adsk.eagle:library:371" deviceset="V+" device=""/>
 <part name="AGND8" library="supply1" library_urn="urn:adsk.eagle:library:371" deviceset="AGND" device=""/>
+<part name="+3V3" library="supply1" library_urn="urn:adsk.eagle:library:371" deviceset="+3V3" device=""/>
+<part name="P+8" library="supply1" library_urn="urn:adsk.eagle:library:371" deviceset="+5V" device=""/>
+<part name="P+9" library="supply1" library_urn="urn:adsk.eagle:library:371" deviceset="+12V" device=""/>
 </parts>
 <sheets>
@@
 <instance part="P+4" gate="1" x="8.89" y="271.78"/>
 <instance part="AGND8" gate="VR1" x="-29.21" y="231.14"/>
+<instance part="+3V3" gate="G$1" x="172.72" y="116.84"/>
+<instance part="P+8" gate="1" x="172.72" y="152.4"/>
+<instance part="P+9" gate="1" x="171.45" y="198.12"/>
 </instances>
 <busses>
@@
 <junction x="203.2" y="246.38"/>
 <junction x="171.45" y="191.77"/>
-<label x="163.83" y="193.04" size="1.778" layer="95"/>
+<pinref part="P+9" gate="1" pin="+12V"/>
+<wire x1="171.45" y1="195.58" x2="171.45" y2="191.77" width="0.1524" layer="91"/>
 </segment>
 </net>
@@
 <wire x1="40.64" y1="111.76" x2="40.64" y2="109.22" width="0.1524" layer="91"/>
 <label x="36.83" y="113.03" size="1.778" layer="95"/>
-</segment>
-</net>
-<net name="+3.3V" class="0">
-<segment>
-<pinref part="C14" gate="G$1" pin="1"/>
-<wire x1="146.05" y1="111.76" x2="160.02" y2="111.76" width="0.1524" layer="91"/>
-<wire x1="160.02" y1="111.76" x2="160.02" y2="107.95" width="0.1524" layer="91"/>
-<pinref part="C13" gate="G$1" pin="1"/>
-<wire x1="146.05" y1="107.95" x2="146.05" y2="111.76" width="0.1524" layer="91"/>
-<pinref part="C15" gate="G$1" pin="1"/>
-<wire x1="160.02" y1="111.76" x2="172.72" y2="111.76" width="0.1524" layer="91"/>
-<wire x1="172.72" y1="111.76" x2="172.72" y2="107.95" width="0.1524" layer="91"/>
-<junction x="160.02" y="111.76"/>
-<label x="165.1" y="113.03" size="1.778" layer="95"/>
 </segment>
 </net>
@@
 <pinref part="+3V2" gate="G$1" pin="+3V3"/>
 </segment>
+<segment>
+<pinref part="C14" gate="G$1" pin="1"/>
+<wire x1="146.05" y1="111.76" x2="160.02" y2="111.76" width="0.1524" layer="91"/>
+<wire x1="160.02" y1="111.76" x2="160.02" y2="107.95" width="0.1524" layer="91"/>
+<pinref part="C13" gate="G$1" pin="1"/>
+<wire x1="146.05" y1="107.95" x2="146.05" y2="111.76" width="0.1524" layer="91"/>
+<pinref part="C15" gate="G$1" pin="1"/>
+<wire x1="160.02" y1="111.76" x2="172.72" y2="111.76" width="0.1524" layer="91"/>
+<wire x1="172.72" y1="111.76" x2="172.72" y2="107.95" width="0.1524" layer="91"/>
+<junction x="160.02" y="111.76"/>
+<pinref part="+3V3" gate="G$1" pin="+3V3"/>
+<wire x1="172.72" y1="114.3" x2="172.72" y2="111.76" width="0.1524" layer="91"/>
+<junction x="172.72" y="111.76"/>
+</segment>
 </net>
 <net name="+5V" class="0">
@@
 <pinref part="C10" gate="G$1" pin="1"/>
 <wire x1="160.02" y1="146.05" x2="172.72" y2="146.05" width="0.1524" layer="91"/>
+<junction x="160.02" y="146.05"/>
+<pinref part="P+8" gate="1" pin="+5V"/>
 <wire x1="172.72" y1="146.05" x2="172.72" y2="142.24" width="0.1524" layer="91"/>
-<junction x="160.02" y="146.05"/>
-<label x="165.1" y="147.32" size="1.778" layer="95"/>
+<wire x1="172.72" y1="149.86" x2="172.72" y2="146.05" width="0.1524" layer="91"/>
+<junction x="172.72" y="146.05"/>
 </segment>
 </net>
@@
 <segment>
 <pinref part="Q2" gate="G$1" pin="G"/>
-<wire x1="-29.21" y1="40.64" x2="-39.37" y2="40.64" width="0.1524" layer="91"/>
+<wire x1="-29.21" y1="40.64" x2="-43.18" y2="40.64" width="0.1524" layer="91"/>
 <label x="-38.1" y="36.83" size="1.778" layer="95"/>
-<pinref part="R3" gate="G$1" pin="1"/>
-<wire x1="-43.18" y1="43.18" x2="-43.18" y2="40.64" width="0.1524" layer="91"/>
-<wire x1="-43.18" y1="40.64" x2="-39.37" y2="40.64" width="0.1524" layer="91"/>
 <junction x="-43.18" y="40.64"/>
 <wire x1="-43.18" y1="40.64" x2="-50.8" y2="40.64" width="0.1524" layer="91"/>
 <pinref part="R7" gate="G$1" pin="2"/>
 <wire x1="-43.18" y1="38.1" x2="-43.18" y2="40.64" width="0.1524" layer="91"/>
-</segment>
-</net>
+<pinref part="R3" gate="G$1" pin="1"/>
+<wire x1="-43.18" y1="43.18" x2="-43.18" y2="40.64" width="0.1524" layer="91"/>
+</segment>
+</net>
