File: Board Template/uwrt/Board Template/uwrt/Battery Balancer/BatteryBalancer.sch (EAGLE design)
At the start: 18 parts, among them P1 39-30-06, P2 39-30-06, P3 39-30-06, P4 39-30-08, P5 39-30-08, P6 39-30-02

Commit message: Changed Battery Balancer
Parts:
- removed P6: 39-30-02, con-molex-mini-fit:39-30-02
Connections:
- removed net LOAD: U$10.LOAD+, U$11.LOAD+, U$8.LOAD+, U$9.LOAD+
- removed net MOTOR_POWER1: P5.1, P5.2, P5.3, P5.4, U$8.LOAD-, U$9.LOAD-
- removed net MOTOR_POWER2: P4.1, P4.2, P4.3, P4.4, U$10.LOAD-, U$11.LOAD-
- removed net SENSOR_SCL: U$1.SENSOR_SCL, U$12.SCL
- removed net SENSOR_SDA: U$1.SENSOR_SDA, U$12.SDA
- new net BALANCED: U$10.LOAD+, U$11.LOAD+, U$2.OUT, U$2.VS, U$3.OUT, U$3.VS, U$4.DRAIN, U$5.DRAIN, U$8.LOAD+, U$9.LOAD+
- new net MOTOR_POWER: P4.1, P4.2, P4.3, P4.4, P5.1, P5.2, P5.3, P5.4, U$10.LOAD-, U$11.LOAD-, U$8.LOAD-, U$9.LOAD-
- net BALANCED_OUT: no longer U$2.OUT, U$2.VS, U$3.OUT, U$3.VS, U$4.DRAIN, U$5.DRAIN
- net KILL_SWITCH: no longer P6.1
- net PORT_CURRENT: no longer U$12.IN0
- net STBD_CURRENT: no longer U$12.IN3
