File: Maelstrom Boards/Backplane/Backplane.sch (EAGLE design)
At the start: 4 parts

Commit message: New schematic template and converter fixes
Connections:
- removed net SPARE10: U$1.SPARE10, U$2.SPARE10, U$3.SPARE10, U$4.SPARE10
- removed net SPARE11: U$1.SPARE11, U$2.SPARE11, U$3.SPARE11, U$4.SPARE11
- removed net SPARE12: U$1.SPARE12, U$2.SPARE12, U$3.SPARE12, U$4.SPARE12
- removed net SPARE13: U$1.SPARE13, U$2.SPARE13, U$3.SPARE13, U$4.SPARE13
- removed net SPARE14: U$1.SPARE14, U$2.SPARE14, U$3.SPARE14, U$4.SPARE14
- removed net SPARE15: U$1.SPARE15, U$2.SPARE15, U$3.SPARE15, U$4.SPARE15
- removed net SPARE16: U$1.SPARE16, U$2.SPARE16, U$3.SPARE16, U$4.SPARE16
- removed net SPARE17: U$1.SPARE17, U$2.SPARE17, U$3.SPARE17, U$4.SPARE17
- removed net SPARE9: U$1.SPARE9, U$2.SPARE9, U$3.SPARE9, U$4.SPARE9
- new net ACOUSTIC_ON/OFF: U$1.ACOUSTIC_ON/OFF, U$2.ACOUSTIC_ON/OFF, U$3.ACOUSTIC_ON/OFF, U$4.ACOUSTIC_ON/OFF
- new net JETSON_ON/OFF: U$1.JETSON_ON/OFF, U$2.JETSON_ON/OFF, U$3.JETSON_ON/OFF, U$4.JETSON_ON/OFF
- new net MOBO_ON/OFF: U$1.MOBO_ON/OFF, U$2.MOBO_ON/OFF, U$3.MOBO_ON/OFF, U$4.MOBO_ON/OFF
Other:
- note added: "Electrical Team"
- note added: "Underwater Robotics Team Ohio State University"

Commit message: Update
Parts:
- added U$5: 5530843-FEMALE, 5530843-6:5530843-FEMALE
Connections:
- net 5V: now also U$5.5V

Commit message: Updated Backplane
Parts:
- removed U$5: 5530843-FEMALE, 5530843-6:5530843-FEMALE
- U$2, U$4: SPICEPREFIX (none) -> X
Connections:
- net 5V: no longer U$5.5V

Commit message: Backplane Update
Parts:
- added P1: 39-30-06_S, con-molex-mini-fit:39-30-06_S
- added P2: 39-30-08_S, con-molex-mini-fit:39-30-08_S
Connections:
- net 3.3V: now also P1-1.P, P2-1.P
- net BOARD_SCL: now also P1-6.P
- net BOARD_SDA: now also P1-3.P
- net GND: now also P1-4.P, P2-5.P
- net KILL_SWITCH: now also P2-2.P
- net SENSOR_SCL: now also P1-5.P
- net SENSOR_SDA: now also P1-2.P
- net SWITCH_1: now also P2-3.P
- net SWITCH_2: now also P2-4.P
- net SWITCH_3: now also P2-6.P
- net SWITCH_4: now also P2-7.P
- net SWITCH_5: now also P2-8.P
Changed lines of the file:
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@@
 <attribute name="SPICEPREFIX" value="X"/>
 </part>
+<part name="P1" library="con-molex-mini-fit" deviceset="39-30-?06?_S" device=""/>
+<part name="P2" library="con-molex-mini-fit" deviceset="39-30-?08?_S" device=""/>
 </parts>
 <sheets>
@@
 <instance part="U$3" gate="G$1" x="127" y="86.36" smashed="yes"/>
 <instance part="U$4" gate="G$1" x="275.59" y="87.63" smashed="yes"/>
+<instance part="P1" gate="-1" x="368.3" y="147.32" smashed="yes">
+<attribute name="VALUE" x="370.84" y="149.86" size="1.778" layer="96" ratio="12" rot="MR0"/>
+<attribute name="PART" x="370.84" y="152.4" size="1.778" layer="95" ratio="12" rot="MR0"/>
+<attribute name="NAME" x="371.475" y="146.685" size="1.778" layer="95" ratio="12"/>
+</instance>
+<instance part="P1" gate="-2" x="368.3" y="142.24" smashed="yes">
+<attribute name="NAME" x="371.475" y="141.605" size="1.778" layer="95" ratio="12"/>
+</instance>
+<instance part="P1" gate="-3" x="368.3" y="137.16" smashed="yes">
+<attribute name="NAME" x="371.475" y="136.525" size="1.778" layer="95" ratio="12"/>
+</instance>
+<instance part="P1" gate="-4" x="368.3" y="132.08" smashed="yes">
+<attribute name="NAME" x="371.475" y="131.445" size="1.778" layer="95" ratio="12"/>
+</instance>
+<instance part="P1" gate="-5" x="368.3" y="127" smashed="yes">
+<attribute name="NAME" x="371.475" y="126.365" size="1.778" layer="95" ratio="12"/>
+</instance>
+<instance part="P1" gate="-6" x="368.3" y="121.92" smashed="yes">
+<attribute name="NAME" x="371.475" y="121.285" size="1.778" layer="95" ratio="12"/>
+</instance>
+<instance part="P2" gate="-1" x="17.78" y="157.48" smashed="yes" rot="MR0">
+<attribute name="VALUE" x="15.24" y="160.02" size="1.778" layer="96" ratio="12"/>
+<attribute name="PART" x="15.24" y="162.56" size="1.778" layer="95" ratio="12"/>
+<attribute name="NAME" x="14.605" y="156.845" size="1.778" layer="95" ratio="12" rot="MR0"/>
+</instance>
+<instance part="P2" gate="-2" x="17.78" y="152.4" smashed="yes" rot="MR0">
+<attribute name="NAME" x="14.605" y="151.765" size="1.778" layer="95" ratio="12" rot="MR0"/>
+</instance>
+<instance part="P2" gate="-3" x="17.78" y="147.32" smashed="yes" rot="MR0">
+<attribute name="NAME" x="14.605" y="146.685" size="1.778" layer="95" ratio="12" rot="MR0"/>
+</instance>
+<instance part="P2" gate="-4" x="17.78" y="142.24" smashed="yes" rot="MR0">
+<attribute name="NAME" x="14.605" y="141.605" size="1.778" layer="95" ratio="12" rot="MR0"/>
+</instance>
+<instance part="P2" gate="-5" x="17.78" y="137.16" smashed="yes" rot="MR0">
+<attribute name="NAME" x="14.605" y="136.525" size="1.778" layer="95" ratio="12" rot="MR0"/>
+</instance>
+<instance part="P2" gate="-6" x="17.78" y="132.08" smashed="yes" rot="MR0">
+<attribute name="NAME" x="14.605" y="131.445" size="1.778" layer="95" ratio="12" rot="MR0"/>
+</instance>
+<instance part="P2" gate="-7" x="17.78" y="127" smashed="yes" rot="MR0">
+<attribute name="NAME" x="14.605" y="126.365" size="1.778" layer="95" ratio="12" rot="MR0"/>
+</instance>
+<instance part="P2" gate="-8" x="17.78" y="121.92" smashed="yes" rot="MR0">
+<attribute name="NAME" x="14.605" y="121.285" size="1.778" layer="95" ratio="12" rot="MR0"/>
+</instance>
 </instances>
 <busses>
@@
 <net name="5V" class="0">
 <segment>
-<wire x1="158.75" y1="313.69" x2="158.75" y2="318.77" width="0.1524" layer="91"/>
-<label x="158.75" y="318.77" size="1.778" layer="95" rot="R90" xref="yes"/>
-</segment>
-<segment>
 <pinref part="U$1" gate="G$1" pin="5V"/>
 <wire x1="68.58" y1="217.17" x2="68.58" y2="226.06" width="0.1524" layer="91"/>
@@
 <label x="224.79" y="116.84" size="1.778" layer="95" rot="R90" xref="yes"/>
 </segment>
+<segment>
+<pinref part="P1" gate="-1" pin="P"/>
+<wire x1="365.76" y1="147.32" x2="355.6" y2="147.32" width="0.1524" layer="91"/>
+<label x="355.6" y="147.32" size="1.778" layer="95" rot="R180" xref="yes"/>
+</segment>
+<segment>
+<pinref part="P2" gate="-1" pin="P"/>
+<wire x1="20.32" y1="157.48" x2="33.02" y2="157.48" width="0.1524" layer="91"/>
+<label x="33.02" y="157.48" size="1.778" layer="95" xref="yes"/>
+</segment>
 </net>
 <net name="PWM_1" class="0">
@@
 <label x="217.17" y="60.96" size="1.778" layer="95" rot="R270" xref="yes"/>
 </segment>
+<segment>
+<pinref part="P1" gate="-3" pin="P"/>
+<wire x1="365.76" y1="137.16" x2="355.6" y2="137.16" width="0.1524" layer="91"/>
+<label x="355.6" y="137.16" size="1.778" layer="95" rot="R180" xref="yes"/>
+</segment>
 </net>
 <net name="BOARD_SCL" class="0">
@@
 <label x="222.25" y="60.96" size="1.778" layer="95" rot="R270" xref="yes"/>
 </segment>
+<segment>
+<pinref part="P1" gate="-6" pin="P"/>
+<wire x1="365.76" y1="121.92" x2="355.6" y2="121.92" width="0.1524" layer="91"/>
+<label x="355.6" y="121.92" size="1.778" layer="95" rot="R180" xref="yes"/>
+</segment>
 </net>
 <net name="SENSOR_SDA" class="0">
@@
 <label x="227.33" y="60.96" size="1.778" layer="95" rot="R270" xref="yes"/>
 </segment>
+<segment>
+<pinref part="P1" gate="-2" pin="P"/>
+<wire x1="365.76" y1="142.24" x2="355.6" y2="142.24" width="0.1524" layer="91"/>
+<label x="355.6" y="142.24" size="1.778" layer="95" rot="R180" xref="yes"/>
+</segment>
 </net>
 <net name="SENSOR_SCL" class="0">
@@
 <label x="232.41" y="60.96" size="1.778" layer="95" rot="R270" xref="yes"/>
 </segment>
+<segment>
+<pinref part="P1" gate="-5" pin="P"/>
+<wire x1="365.76" y1="127" x2="355.6" y2="127" width="0.1524" layer="91"/>
+<label x="355.6" y="127" size="1.778" layer="95" rot="R180" xref="yes"/>
+</segment>
 </net>
 <net name="KILL_SWITCH" class="0">
@@
 <label x="242.57" y="60.96" size="1.778" layer="95" rot="R270" xref="yes"/>
 </segment>
+<segment>
+<pinref part="P2" gate="-2" pin="P"/>
+<wire x1="20.32" y1="152.4" x2="33.02" y2="152.4" width="0.1524" layer="91"/>
+<label x="33.02" y="152.4" size="1.778" layer="95" xref="yes"/>
+</segment>
 </net>
 <net name="SWITCH_1" class="0">
@@
 <label x="247.65" y="60.96" size="1.778" layer="95" rot="R270" xref="yes"/>
 </segment>
+<segment>
+<pinref part="P2" gate="-3" pin="P"/>
+<wire x1="20.32" y1="147.32" x2="33.02" y2="147.32" width="0.1524" layer="91"/>
+<label x="33.02" y="147.32" size="1.778" layer="95" xref="yes"/>
+</segment>
 </net>
 <net name="SWITCH_2" class="0">
@@
 <label x="252.73" y="60.96" size="1.778" layer="95" rot="R270" xref="yes"/>
 </segment>
+<segment>
+<pinref part="P2" gate="-4" pin="P"/>
+<wire x1="20.32" y1="142.24" x2="33.02" y2="142.24" width="0.1524" layer="91"/>
+<label x="33.02" y="142.24" size="1.778" layer="95" xref="yes"/>
+</segment>
 </net>
 <net name="SWITCH_3" class="0">
@@
 <label x="257.81" y="60.96" size="1.778" layer="95" rot="R270" xref="yes"/>
 </segment>
+<segment>
+<pinref part="P2" gate="-6" pin="P"/>
+<wire x1="20.32" y1="132.08" x2="33.02" y2="132.08" width="0.1524" layer="91"/>
+<label x="33.02" y="132.08" size="1.778" layer="95" xref="yes"/>
+</segment>
 </net>
 <net name="SWITCH_4" class="0">
@@
 <label x="262.89" y="60.96" size="1.778" layer="95" rot="R270" xref="yes"/>
 </segment>
+<segment>
+<pinref part="P2" gate="-7" pin="P"/>
+<wire x1="20.32" y1="127" x2="33.02" y2="127" width="0.1524" layer="91"/>
+<label x="33.02" y="127" size="1.778" layer="95" xref="yes"/>
+</segment>
 </net>
 <net name="SWITCH_5" class="0">
@@
 <label x="267.97" y="60.96" size="1.778" layer="95" rot="R270" xref="yes"/>
 </segment>
+<segment>
+<pinref part="P2" gate="-8" pin="P"/>
+<wire x1="20.32" y1="121.92" x2="33.02" y2="121.92" width="0.1524" layer="91"/>
+<label x="33.02" y="121.92" size="1.778" layer="95" xref="yes"/>
+</segment>
 </net>
 <net name="GND" class="0">
@@
 <label x="278.13" y="60.96" size="1.778" layer="95" rot="R270" xref="yes"/>
 </segment>
+<segment>
+<pinref part="P1" gate="-4" pin="P"/>
+<wire x1="365.76" y1="132.08" x2="355.6" y2="132.08" width="0.1524" layer="91"/>
+<label x="355.6" y="132.08" size="1.778" layer="95" rot="R180" xref="yes"/>
+</segment>
+<segment>
+<pinref part="P2" gate="-5" pin="P"/>
+<wire x1="20.32" y1="137.16" x2="33.02" y2="137.16" width="0.1524" layer="91"/>
+<label x="33.02" y="137.16" size="1.778" layer="95" xref="yes"/>
+</segment>
 </net>

Commit message: Updated Backplane
Parts:
- removed P1: 39-30-06_S, con-molex-mini-fit:39-30-06_S
- removed P2: 39-30-08_S, con-molex-mini-fit:39-30-08_S
- added P3: 39-30-04_S, con-molex-mini-fit:39-30-04_S
- added SWITCH_CONNECTOR: 39-30-08_S, con-molex-mini-fit:39-30-08_S
- added U$5: 929870-01-09_1, 3M_929852_Connector:929870-01-09_1
- added U$6: 929870-01-09_2, 3M_929852_Connector:929870-01-09_2
- added U$7: 929870-01-09_3, 3M_929852_Connector:929870-01-09_3
- added U$8: 929870-01-09_4, 3M_929852_Connector:929870-01-09_4
Connections:
- removed net BOARD_SCL: P1-6.P, U$1.BOARD_SCL, U$2.BOARD_SCL, U$3.BOARD_SCL, U$4.BOARD_SCL
- removed net BOARD_SDA: P1-3.P, U$1.BOARD_SDA, U$2.BOARD_SDA, U$3.BOARD_SDA, U$4.BOARD_SDA
- removed net SENSOR_SCL: P1-5.P, U$1.SENSOR_SCL, U$2.SENSOR_SCL, U$3.SENSOR_SCL, U$4.SENSOR_SCL
- removed net SENSOR_SDA: P1-2.P, U$1.SENSOR_SDA, U$2.SENSOR_SDA, U$3.SENSOR_SDA, U$4.SENSOR_SDA
- new net BACKPLANE_SCL: U$1.BACKPLANE_SCL, U$2.BACKPLANE_SCL, U$3.BACKPLANE_SCL, U$4.BACKPLANE_SCL, U$8.BACKPLANE_SCL
- new net BACKPLANE_SDA: U$1.BACKPLANE_SDA, U$2.BACKPLANE_SDA, U$3.BACKPLANE_SDA, U$4.BACKPLANE_SDA, U$8.BACKPLANE_SDA
- new net ROBOT_SCL: P3-4.P, U$1.ROBOT_SCL, U$2.ROBOT_SCL, U$3.ROBOT_SCL, U$4.ROBOT_SCL, U$8.ROBOT_SCL
- new net ROBOT_SDA: P3-2.P, U$1.ROBOT_SDA, U$2.ROBOT_SDA, U$3.ROBOT_SDA, U$4.ROBOT_SDA, U$8.ROBOT_SDA
- net 12V_ON/OFF: now also U$7.12V_ON/OFF
- net 3.3V: now also P3-1.P, U$8.3.3V; no longer P1-1.P, P2-1.P
- net 3.3V_ON/OFF: now also U$7.3.3V_ON/OFF
- net 5V: now also SWITCH_CONNECTOR-1.P, U$8.5V
- net 5V_ON/OFF: now also U$7.5V-ON/OFF
- net ACOUSTIC_ON/OFF: now also U$7.ACOUSTIC_ON/OFF
- net GND: now also P3-3.P, SWITCH_CONNECTOR-5.P, U$7.GND, U$8.GND; no longer P1-4.P, P2-5.P
- net JETSON_ON/OFF: now also U$7.JETSON_ON/OFF
- net KILL_SWITCH: now also SWITCH_CONNECTOR-2.P, U$5.KILL_SWITCH; no longer P2-2.P
- net MOBO_ON/OFF: now also U$7.MOBO_ON/OFF
- net PWM_1: now also U$6.PWM_1
- net PWM_2: now also U$6.PWM_2
- net PWM_3: now also U$6.PWM_3
- net PWM_4: now also U$6.PWM_4
- net PWM_5: now also U$6.PWM_5
- net PWM_6: now also U$6.PWM_6
- net PWM_7: now also U$6.PWM_7
- net PWM_8: now also U$6.PWM_8
- net SPARE1: now also U$7.SPARE1
- net SPARE2: now also U$6.SPARE2
- net SPARE3: now also U$8.SPARE3
- net SPARE4: now also U$8.SPARE4
- net SPARE5: now also U$5.SPARE5
- net SPARE6: now also U$5.SPARE6
- net SPARE7: now also U$5.SPARE7
- net SPARE8: now also U$7.SPARE8
- net SWITCH_1: now also SWITCH_CONNECTOR-3.P, U$5.SWITCH_1; no longer P2-3.P
- net SWITCH_2: now also SWITCH_CONNECTOR-4.P, U$5.SWITCH_2; no longer P2-4.P
- net SWITCH_3: now also SWITCH_CONNECTOR-6.P, U$5.SWITCH_3; no longer P2-6.P
- net SWITCH_4: now also SWITCH_CONNECTOR-7.P, U$5.SWITCH_4; no longer P2-7.P
- net SWITCH_5: now also SWITCH_CONNECTOR-8.P, U$5.SWITCH_5; no longer P2-8.P
