File: Maelstrom Boards/Backplane/Backplane.brd (EAGLE design)
At the start: 254 x 101.7 mm, 29 parts, among them P1 39-30-02?_S, P3 39-30-04?_S

Commit message: Final changes before order
Parts:
- R1, R10, R11, R12, R13, R14, R2, R3, R4, R5, R6, R7, R8, R9: value (none) -> 10k
Changed lines of the file:
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@@
 <attribute name="VALUE" x="0.0889" y="85.979" size="1.016" layer="27" ratio="10"/>
 </element>
-<element name="R1" library="rcl" library_urn="urn:adsk.eagle:library:334" package="R0603" package3d_urn="urn:adsk.eagle:package:23555/2" value="" x="204.597" y="50.038" smashed="yes" rot="R270">
+<element name="R1" library="rcl" library_urn="urn:adsk.eagle:library:334" package="R0603" package3d_urn="urn:adsk.eagle:package:23555/2" value="10k" x="204.597" y="50.038" smashed="yes" rot="R270">
 <attribute name="NAME" x="205.232" y="50.673" size="1.27" layer="25" rot="R270"/>
 <attribute name="SPICEPREFIX" value="R" x="204.597" y="50.038" size="1.778" layer="27" rot="R270" display="off"/>
 <attribute name="VALUE" x="202.692" y="50.673" size="1.27" layer="27" rot="R270"/>
 </element>
-<element name="R2" library="rcl" library_urn="urn:adsk.eagle:library:334" package="R0603" package3d_urn="urn:adsk.eagle:package:23555/2" value="" x="208.026" y="50.038" smashed="yes" rot="R270">
+<element name="R2" library="rcl" library_urn="urn:adsk.eagle:library:334" package="R0603" package3d_urn="urn:adsk.eagle:package:23555/2" value="10k" x="208.026" y="50.038" smashed="yes" rot="R270">
 <attribute name="NAME" x="208.661" y="50.673" size="1.27" layer="25" rot="R270"/>
 <attribute name="SPICEPREFIX" value="R" x="208.026" y="50.038" size="1.778" layer="27" rot="R270" display="off"/>
 <attribute name="VALUE" x="206.121" y="50.673" size="1.27" layer="27" rot="R270"/>
 </element>
-<element name="R3" library="rcl" library_urn="urn:adsk.eagle:library:334" package="R0603" package3d_urn="urn:adsk.eagle:package:23555/2" value="" x="211.582" y="50.038" smashed="yes" rot="R270">
+<element name="R3" library="rcl" library_urn="urn:adsk.eagle:library:334" package="R0603" package3d_urn="urn:adsk.eagle:package:23555/2" value="10k" x="211.582" y="50.038" smashed="yes" rot="R270">
 <attribute name="NAME" x="212.217" y="50.673" size="1.27" layer="25" rot="R270"/>
 <attribute name="SPICEPREFIX" value="R" x="211.582" y="50.038" size="1.778" layer="27" rot="R270" display="off"/>
 <attribute name="VALUE" x="209.677" y="50.673" size="1.27" layer="27" rot="R270"/>
 </element>
-<element name="R4" library="rcl" library_urn="urn:adsk.eagle:library:334" package="R0603" package3d_urn="urn:adsk.eagle:package:23555/2" value="" x="215.265" y="50.038" smashed="yes" rot="R270">
+<element name="R4" library="rcl" library_urn="urn:adsk.eagle:library:334" package="R0603" package3d_urn="urn:adsk.eagle:package:23555/2" value="10k" x="215.265" y="50.038" smashed="yes" rot="R270">
 <attribute name="NAME" x="215.9" y="50.673" size="1.27" layer="25" rot="R270"/>
 <attribute name="SPICEPREFIX" value="R" x="215.265" y="50.038" size="1.778" layer="27" rot="R270" display="off"/>
 <attribute name="VALUE" x="213.36" y="50.673" size="1.27" layer="27" rot="R270"/>
 </element>
-<element name="R5" library="rcl" library_urn="urn:adsk.eagle:library:334" package="R0603" package3d_urn="urn:adsk.eagle:package:23555/2" value="" x="219.075" y="50.038" smashed="yes" rot="R270">
+<element name="R5" library="rcl" library_urn="urn:adsk.eagle:library:334" package="R0603" package3d_urn="urn:adsk.eagle:package:23555/2" value="10k" x="219.075" y="50.038" smashed="yes" rot="R270">
 <attribute name="NAME" x="219.71" y="50.673" size="1.27" layer="25" rot="R270"/>
 <attribute name="SPICEPREFIX" value="R" x="219.075" y="50.038" size="1.778" layer="27" rot="R270" display="off"/>
 <attribute name="VALUE" x="217.17" y="50.673" size="1.27" layer="27" rot="R270"/>
 </element>
-<element name="R6" library="rcl" library_urn="urn:adsk.eagle:library:334" package="R0603" package3d_urn="urn:adsk.eagle:package:23555/2" value="" x="222.758" y="50.038" smashed="yes" rot="R270">
+<element name="R6" library="rcl" library_urn="urn:adsk.eagle:library:334" package="R0603" package3d_urn="urn:adsk.eagle:package:23555/2" value="10k" x="222.758" y="50.038" smashed="yes" rot="R270">
 <attribute name="NAME" x="223.393" y="50.673" size="1.27" layer="25" rot="R270"/>
 <attribute name="SPICEPREFIX" value="R" x="222.758" y="50.038" size="1.778" layer="27" rot="R270" display="off"/>
 <attribute name="VALUE" x="220.853" y="50.673" size="1.27" layer="27" rot="R270"/>
 </element>
-<element name="R7" library="rcl" library_urn="urn:adsk.eagle:library:334" package="R0603" package3d_urn="urn:adsk.eagle:package:23555/2" value="" x="226.187" y="50.038" smashed="yes" rot="R270">
+<element name="R7" library="rcl" library_urn="urn:adsk.eagle:library:334" package="R0603" package3d_urn="urn:adsk.eagle:package:23555/2" value="10k" x="226.187" y="50.038" smashed="yes" rot="R270">
 <attribute name="NAME" x="226.822" y="50.673" size="1.27" layer="25" rot="R270"/>
 <attribute name="SPICEPREFIX" value="R" x="226.187" y="50.038" size="1.778" layer="27" rot="R270" display="off"/>
 <attribute name="VALUE" x="224.282" y="50.673" size="1.27" layer="27" rot="R270"/>
 </element>
-<element name="R8" library="rcl" library_urn="urn:adsk.eagle:library:334" package="R0603" package3d_urn="urn:adsk.eagle:package:23555/2" value="" x="229.743" y="50.038" smashed="yes" rot="R270">
+<element name="R8" library="rcl" library_urn="urn:adsk.eagle:library:334" package="R0603" package3d_urn="urn:adsk.eagle:package:23555/2" value="10k" x="229.743" y="50.038" smashed="yes" rot="R270">
 <attribute name="NAME" x="230.378" y="50.673" size="1.27" layer="25" rot="R270"/>
 <attribute name="SPICEPREFIX" value="R" x="229.743" y="50.038" size="1.778" layer="27" rot="R270" display="off"/>
 <attribute name="VALUE" x="227.838" y="50.673" size="1.27" layer="27" rot="R270"/>
 </element>
-<element name="R9" library="rcl" library_urn="urn:adsk.eagle:library:334" package="R0603" package3d_urn="urn:adsk.eagle:package:23555/2" value="" x="12.319" y="11.176" smashed="yes" rot="R180">
+<element name="R9" library="rcl" library_urn="urn:adsk.eagle:library:334" package="R0603" package3d_urn="urn:adsk.eagle:package:23555/2" value="10k" x="12.319" y="11.176" smashed="yes" rot="R180">
 <attribute name="NAME" x="12.954" y="10.541" size="1.27" layer="25" rot="R180"/>
 <attribute name="SPICEPREFIX" value="R" x="12.319" y="11.176" size="1.778" layer="27" rot="R180" display="off"/>
 <attribute name="VALUE" x="12.954" y="13.081" size="1.27" layer="27" rot="R180"/>
 </element>
-<element name="R10" library="rcl" library_urn="urn:adsk.eagle:library:334" package="R0603" package3d_urn="urn:adsk.eagle:package:23555/2" value="" x="12.319" y="14.605" smashed="yes" rot="R180">
+<element name="R10" library="rcl" library_urn="urn:adsk.eagle:library:334" package="R0603" package3d_urn="urn:adsk.eagle:package:23555/2" value="10k" x="12.319" y="14.605" smashed="yes" rot="R180">
 <attribute name="NAME" x="-134.366" y="-67.056" size="1.27" layer="25" rot="R270"/>
 <attribute name="SPICEPREFIX" value="R" x="12.319" y="14.605" size="1.778" layer="27" rot="R180" display="off"/>
 <attribute name="VALUE" x="12.954" y="16.51" size="1.27" layer="27" rot="R180"/>
 </element>
-<element name="R11" library="rcl" library_urn="urn:adsk.eagle:library:334" package="R0603" package3d_urn="urn:adsk.eagle:package:23555/2" value="" x="12.319" y="17.653" smashed="yes" rot="R180">
+<element name="R11" library="rcl" library_urn="urn:adsk.eagle:library:334" package="R0603" package3d_urn="urn:adsk.eagle:package:23555/2" value="10k" x="12.319" y="17.653" smashed="yes" rot="R180">
 <attribute name="NAME" x="12.954" y="17.018" size="1.27" layer="25" rot="R180"/>
 <attribute name="SPICEPREFIX" value="R" x="12.319" y="17.653" size="1.778" layer="27" rot="R180" display="off"/>
 <attribute name="VALUE" x="12.954" y="19.558" size="1.27" layer="27" rot="R180"/>
 </element>
-<element name="R12" library="rcl" library_urn="urn:adsk.eagle:library:334" package="R0603" package3d_urn="urn:adsk.eagle:package:23555/2" value="" x="12.319" y="20.828" smashed="yes" rot="R180">
+<element name="R12" library="rcl" library_urn="urn:adsk.eagle:library:334" package="R0603" package3d_urn="urn:adsk.eagle:package:23555/2" value="10k" x="12.319" y="20.828" smashed="yes" rot="R180">
 <attribute name="NAME" x="12.954" y="20.193" size="1.27" layer="25" rot="R180"/>
 <attribute name="SPICEPREFIX" value="R" x="12.319" y="20.828" size="1.778" layer="27" rot="R180" display="off"/>
 <attribute name="VALUE" x="12.954" y="22.733" size="1.27" layer="27" rot="R180"/>
 </element>
-<element name="R13" library="rcl" library_urn="urn:adsk.eagle:library:334" package="R0603" package3d_urn="urn:adsk.eagle:package:23555/2" value="" x="12.319" y="23.876" smashed="yes" rot="R180">
+<element name="R13" library="rcl" library_urn="urn:adsk.eagle:library:334" package="R0603" package3d_urn="urn:adsk.eagle:package:23555/2" value="10k" x="12.319" y="23.876" smashed="yes" rot="R180">
 <attribute name="NAME" x="12.954" y="23.241" size="1.27" layer="25" rot="R180"/>
 <attribute name="SPICEPREFIX" value="R" x="12.319" y="23.876" size="1.778" layer="27" rot="R180" display="off"/>
 <attribute name="VALUE" x="12.954" y="25.781" size="1.27" layer="27" rot="R180"/>
 </element>
-<element name="R14" library="rcl" library_urn="urn:adsk.eagle:library:334" package="R0603" package3d_urn="urn:adsk.eagle:package:23555/2" value="" x="12.319" y="27.051" smashed="yes" rot="R180">
+<element name="R14" library="rcl" library_urn="urn:adsk.eagle:library:334" package="R0603" package3d_urn="urn:adsk.eagle:package:23555/2" value="10k" x="12.319" y="27.051" smashed="yes" rot="R180">
 <attribute name="NAME" x="12.954" y="26.416" size="1.27" layer="25" rot="R180"/>
 <attribute name="SPICEPREFIX" value="R" x="12.319" y="27.051" size="1.778" layer="27" rot="R180" display="off"/>
