File: Maelstrom Boards/CoProcessor/CoProcessorSP20.sch (EAGLE design)
At the start: 77 parts, among them J1 USB_MINI-B_SMT, P1 RB1-125BAG1A, Q1 310mA/60V/1.6Ω, Q2 310mA/60V/1.6Ω, Q3 310mA/60V/1.6Ω, Q4 310mA/60V/1.6Ω, Q5 310mA/60V/1.6Ω, Q6 310mA/60V/1.6Ω, Q7 310mA/60V/1.6Ω, Q8 310mA/60V/1.6Ω, U1 W5500, U2 STM32F405RGT6, Y1 12MHz, Y2 25MHz, Y3 32.768kHz

Commit message: coprocessor changes
Parts:
- removed J2: (no value), SparkFun-Connectors:CONN_04
- added JP1: (no value), pinhead:PINHD-2X10
Connections:
- net +3V3: now also JP1.19; no longer J2.4
- net GND: now also JP1.20; no longer J2.1
- net SWCLK: now also JP1.9; no longer J2.2
- net SWDIO: now also JP1.7; no longer J2.3
Changed lines of the file:
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@@
 <part name="R32" library="rcl" library_urn="urn:adsk.eagle:library:334" deviceset="R-US_" device="R0603" package3d_urn="urn:adsk.eagle:package:23555/2" value="5"/>
 <part name="+3V22" library="supply1" library_urn="urn:adsk.eagle:library:371" deviceset="+3V3" device=""/>
-<part name="J2" library="SparkFun-Connectors" library_urn="urn:adsk.eagle:library:513" deviceset="CONN_04" device="" package3d_urn="urn:adsk.eagle:package:38085/1"/>
-<part name="+3V23" library="supply1" library_urn="urn:adsk.eagle:library:371" deviceset="+3V3" device=""/>
-<part name="GND19" library="supply1" library_urn="urn:adsk.eagle:library:371" deviceset="GND" device=""/>
 <part name="C21" library="rcl" library_urn="urn:adsk.eagle:library:334" deviceset="C-EU" device="C0603" package3d_urn="urn:adsk.eagle:package:23616/2" value="0.1uF"/>
 <part name="C22" library="rcl" library_urn="urn:adsk.eagle:library:334" deviceset="C-EU" device="C0603" package3d_urn="urn:adsk.eagle:package:23616/2" value="0.1uF"/>
@@
 <part name="R5" library="rcl" library_urn="urn:adsk.eagle:library:334" deviceset="R-US_" device="R0603" package3d_urn="urn:adsk.eagle:package:23555/2" value="65"/>
 <part name="R6" library="rcl" library_urn="urn:adsk.eagle:library:334" deviceset="R-US_" device="R0603" package3d_urn="urn:adsk.eagle:package:23555/2" value="65"/>
+<part name="JP1" library="pinhead" library_urn="urn:adsk.eagle:library:325" deviceset="PINHD-2X10" device="" package3d_urn="urn:adsk.eagle:package:22405/2"/>
+<part name="+3V2" library="supply1" library_urn="urn:adsk.eagle:library:371" deviceset="+3V3" device=""/>
+<part name="GND20" library="supply1" library_urn="urn:adsk.eagle:library:371" deviceset="GND" device=""/>
 </parts>
 <sheets>
@@
 <attribute name="VALUE" x="142.24" y="167.64" size="1.778" layer="96" rot="R90"/>
 </instance>
-<instance part="J2" gate="G$1" x="91.44" y="109.22" smashed="yes">
-<attribute name="VALUE" x="86.36" y="101.854" size="1.778" layer="96" font="vector"/>
-<attribute name="NAME" x="86.36" y="117.348" size="1.778" layer="95" font="vector"/>
+<instance part="JP1" gate="A" x="90.805" y="110.49"/>
+<instance part="+3V2" gate="G$1" x="78.105" y="102.87" smashed="yes">
+<attribute name="VALUE" x="75.565" y="97.79" size="1.778" layer="96" rot="R90"/>
 </instance>
-<instance part="+3V23" gate="G$1" x="104.14" y="119.38" smashed="yes">
-<attribute name="VALUE" x="101.6" y="114.3" size="1.778" layer="96" rot="R90"/>
-</instance>
-<instance part="GND19" gate="1" x="104.14" y="101.6" smashed="yes">
-<attribute name="VALUE" x="101.6" y="99.06" size="1.778" layer="96"/>
+<instance part="GND20" gate="1" x="106.68" y="92.075" smashed="yes">
+<attribute name="VALUE" x="104.14" y="89.535" size="1.778" layer="96"/>
 </instance>
 </instances>
@@
 </segment>
 <segment>
-<pinref part="J2" gate="G$1" pin="4"/>
-<wire x1="96.52" y1="114.3" x2="104.14" y2="114.3" width="0.1524" layer="91"/>
-<wire x1="104.14" y1="114.3" x2="104.14" y2="116.84" width="0.1524" layer="91"/>
-<pinref part="+3V23" gate="G$1" pin="+3V3"/>
+<pinref part="JP1" gate="A" pin="19"/>
+<wire x1="88.265" y1="97.79" x2="78.105" y2="97.79" width="0.1524" layer="91"/>
+<wire x1="78.105" y1="97.79" x2="78.105" y2="100.33" width="0.1524" layer="91"/>
+<pinref part="+3V2" gate="G$1" pin="+3V3"/>
 </segment>
 </net>
@@
 </segment>
 <segment>
-<pinref part="J2" gate="G$1" pin="1"/>
-<wire x1="96.52" y1="106.68" x2="104.14" y2="106.68" width="0.1524" layer="91"/>
-<wire x1="104.14" y1="106.68" x2="104.14" y2="104.14" width="0.1524" layer="91"/>
-<pinref part="GND19" gate="1" pin="GND"/>
+<pinref part="JP1" gate="A" pin="20"/>
+<wire x1="95.885" y1="97.79" x2="106.68" y2="97.79" width="0.1524" layer="91"/>
+<wire x1="106.68" y1="97.79" x2="106.68" y2="94.615" width="0.1524" layer="91"/>
+<pinref part="GND20" gate="1" pin="GND"/>
 </segment>
 </net>
@@
 <net name="SWDIO" class="0">
 <segment>
-<pinref part="J2" gate="G$1" pin="3"/>
-<wire x1="96.52" y1="111.76" x2="111.76" y2="111.76" width="0.1524" layer="91"/>
-<label x="111.76" y="111.76" size="1.778" layer="95" xref="yes"/>
+<label x="78.74" y="113.03" size="1.778" layer="95" rot="R180" xref="yes"/>
+<pinref part="JP1" gate="A" pin="7"/>
+<wire x1="88.265" y1="113.03" x2="78.74" y2="113.03" width="0.1524" layer="91"/>
 </segment>
 </net>
 <net name="SWCLK" class="0">
 <segment>
-<pinref part="J2" gate="G$1" pin="2"/>
-<wire x1="96.52" y1="109.22" x2="109.22" y2="109.22" width="0.1524" layer="91"/>
-<wire x1="109.22" y1="109.22" x2="109.22" y2="106.68" width="0.1524" layer="91"/>
-<wire x1="109.22" y1="106.68" x2="111.76" y2="106.68" width="0.1524" layer="91"/>
-<label x="111.76" y="106.68" size="1.778" layer="95" xref="yes"/>
-</segment>
-</net>
+<wire x1="81.28" y1="109.22" x2="76.835" y2="109.22" width="0.1524" layer="91"/>
+<label x="76.835" y="109.22" size="1.778" layer="95" rot="R180" xref="yes"/>
+<wire x1="81.28" y1="109.22" x2="81.28" y2="110.49" width="0.1524" layer="91"/>
+<pinref part="JP1" gate="A" pin="9"/>
+<wire x1="81.28" y1="110.49" x2="88.265" y2="110.49" width="0.1524" layer="91"/>
+</segment>
+</net>
