File: Maelstrom Boards/CoProcessor/CoProcessorSP20.brd (EAGLE design)
At the start: 101.6 x 101.6 mm, 77 parts, among them J1 USB_MINI-B_SMT, P1 RB1-125BAG1A, Q1 310mA/60V/1.6Ω, Q2 310mA/60V/1.6Ω, Q3 310mA/60V/1.6Ω, Q4 310mA/60V/1.6Ω, Q5 310mA/60V/1.6Ω, Q6 310mA/60V/1.6Ω, Q7 310mA/60V/1.6Ω, Q8 310mA/60V/1.6Ω, U1 W5500, U2 STM32F405RGT6, Y1 12MHz, Y2 25MHz, Y3 32.768kHz

Commit message: I forgot to commit these before for the copro
Parts:
- removed J2: (no value), SparkFun-Connectors:1X04
- added SWDIO/SWDCLK/RESET: (no value), SparkFun-Connectors:2X10
- moved C9 12.4 mm to (25.0, 73.4), turned to 180 degrees
- moved C10 10.7 mm to (30.9, 82.6), flipped to the bottom, turned to 0 degrees
- moved R29 7.99 mm to (34.2, 80.2), flipped to the bottom
- moved P1 6.00 mm to (14.5, 81.8)
- moved C20 5.97 mm to (41.5, 38.5), turned to 180 degrees
- moved R11 5.56 mm to (87.3, 84.4)
- moved R20 4.88 mm to (87.4, 78.0)
- moved C11 4.62 mm to (33.6, 77.9)
- moved C15 4.52 mm to (42.7, 42.6), turned to 180 degrees
- moved R25 3.89 mm to (28.6, 88.5)
- moved R21 3.74 mm to (31.5, 73.3), turned to 90 degrees
- moved C13 3.36 mm to (40.0, 51.1), flipped to the bottom, turned to 90 degrees
- moved R12 3.31 mm to (91.8, 78.9)
- moved R13 3.26 mm to (94.1, 79.8)
- moved C14 2.91 mm to (40.5, 54.5), flipped to the bottom, turned to 0 degrees
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Connections:
- net +3V3: now also SWDIO/SWDCLK/RESET.1, SWDIO/SWDCLK/RESET.2; no longer J2.4
- net GND: now also SWDIO/SWDCLK/RESET.10, SWDIO/SWDCLK/RESET.12, SWDIO/SWDCLK/RESET.14, SWDIO/SWDCLK/RESET.16, SWDIO/SWDCLK/RESET.18, SWDIO/SWDCLK/RESET.20, SWDIO/SWDCLK/RESET.4, SWDIO/SWDCLK/RESET.6, SWDIO/SWDCLK/RESET.8; no longer J2.1
- net SWCLK: now also SWDIO/SWDCLK/RESET.9; no longer J2.2
- net SWDIO: now also SWDIO/SWDCLK/RESET.7; no longer J2.3
Routing:
- net GND: track 149.8 -> 103.0 mm, vias 24 -> 29
- net N$18: track 19.3 -> 8.68 mm, vias 2 -> 1
- net N$17: track 29.6 -> 21.0 mm
- net N$16: track 27.2 -> 19.4 mm
- net 5V_CNTRL: track 104.6 -> 97.5 mm, vias 5 -> 7
- net +3V3: track 351.2 -> 357.6 mm, vias 13 -> 12
- net N$26: track 3.21 -> 9.28 mm
- net N$21: track 22.4 -> 16.5 mm
- net N$2: track 12.5 -> 7.72 mm
- net N$14: track 4.53 -> 8.44 mm
- net PLTA_CNTRL: track 55.3 -> 51.5 mm
- net N$20: track 28.9 -> 26.3 mm
- net SWDIO: track 44.2 -> 46.9 mm
- net N$29: track 10.2 -> 7.51 mm, vias 0 -> 1
- net N$19: track 12.6 -> 10.0 mm, vias 0 -> 1
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