File: Maelstrom Boards/Actuator/Actuator.brd (EAGLE design)
At the start: 101.6 x 101.6 mm, 65 parts, among them J1 USB_MINI-B_SMT, P2 39-30-16?, U2 STM32F405RGT6, Y1 12MHz, Y3 32.768kHz

Commit message: Actuator new
Parts:
- removed C1, C6: 30pF, rcl:C0603
- removed C24: 220nF, rcl:C0603
- removed C25: 100nF, rcl:C0603
- removed Q16: (no value), crystal:HC49UP
- removed R42, R8: 10K, rcl:R0603
- removed R5: 100K, rcl:R0603
- removed R6: 5, rcl:R0603
- removed U$5: 18F4550, 18f4550:TQFP-44A-44
- added LED1, LED15, LED18, LED19, LED20, LED21, LED22, LED23, LED24, LED25, LED26, LED27: (no value), led:CHIPLED_0603
- added R14, R18, R19, R22, R23, R24, R25, R26, R28: 100, resistor:R0805
- added R15: 220, resistor:R0805
- added R16: 680, resistor:R0805
- added R17: 1.5k, resistor:R0805
- moved J2 321.8 mm to (48.8, 86.3), turned to 180 degrees
- moved R1 313.7 mm to (15.0, 86.2), turned to 270 degrees
- moved R13 310.9 mm to (18.6, 88.4), turned to 270 degrees
- moved R11 310.0 mm to (10.5, 87.7), turned to 270 degrees
- moved J1 307.9 mm to (14.3, 95.4), turned to 270 degrees
- moved R2 305.8 mm to (10.5, 83.4), turned to 270 degrees
- moved C3 295.9 mm to (34.1, 91.7), flipped to the bottom, turned to 180 degrees
- moved C9 295.5 mm to (37.5, 95.8), turned to 180 degrees
- moved R27 294.6 mm to (29.2, 91.7), turned to 180 degrees
- moved Y3 293.4 mm to (39.2, 90.7), turned to 270 degrees
- moved S2 289.3 mm to (46.9, 95.8), flipped to the bottom, turned to 90 degrees
- moved C2 287.0 mm to (26.2, 89.5), flipped to the bottom, turned to 270 degrees
- moved C13 286.4 mm to (34.6, 87.7), turned to 90 degrees
- moved Y1 285.8 mm to (25.6, 95.6), flipped to the bottom, turned to 180 degrees
- moved R30 282.7 mm to (31.5, 79.2), flipped to the bottom
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Connections:
- removed net !MCLR!: U$5.18
- removed net N$32: C24.1, U$5.37
- removed net N$33: R42.1, U$5.15
- removed net PGC: U$5.16
- removed net PGD: U$5.17
- removed net PWM: U$5.35
- removed net USB+: U$5.43
- removed net USB-: U$5.42
- new net EXTRA1: U$1.28, U2.52
- new net EXTRA2: U$1.33, U2.53
- new net EXTRA3: U$1.34, U2.54
- new net EXTRA4: U$1.43, U2.51
- new net EXTRA5: U$1.36, U2.56
- new net EXTRA6: U$1.35, U2.55
- new net LED1: LED20.A, U2.20
- new net LED2: LED21.A, U2.21
- new net LED3: LED22.A, U2.22
- new net LED4: LED23.A, U2.23
- new net LED5: LED24.A, U2.24
- new net LED6: LED25.A, U2.25
- new net LED7: LED26.A, U2.26
- new net LED8: LED27.A, U2.27
- new net N$12: LED15.C, R15.2
- new net N$13: LED18.C, R16.2
- new net N$16: LED20.C, R18.2
- new net N$17: LED21.C, R19.2
- new net N$18: LED22.C, R22.2
- new net N$19: LED23.C, R23.2
- new net N$21: LED24.C, R24.2
- new net SMBA: U2.57
- new net SWD_CLK: J2.2, U2.49
- new net SWD_IO: J2.3, U2.46
- net +12V: now also LED18.A
- net +24V: now also LED19.A; no longer R5.1
- net +3V3: now also J2.4, LED1.A; no longer C25.1, U$5.28, U$5.7
- net +5V: now also LED15.A
- net AGND: now also J2.1, R14.1, R15.1, R16.1, R17.1, R18.1, R19.1, R22.1, R23.1, R24.1, R25.1, R26.1, R28.1; no longer C1.2, C24.2, C25.2, C6.2, R42.2, R8.2, U$5.29, U$5.6
- net ARM_TORPEDO: no longer U$5.10
- net COIL_1_GATE: no longer U$5.38
- net COIL_2_GATE: no longer U$5.39
- net COIL_3_GATE: no longer U$5.40
- net COIL_4_GATE: no longer U$5.41
- net COIL_5_GATE: no longer U$5.2
- net COIL_S_GATE: no longer U$5.3
- net DROPPER1_GATE: no longer U$5.4
- net DROPPER2_GATE: no longer U$5.5
- net N$15: now also LED19.C, R17.2; no longer R6.2
- net N$22: now also LED25.C, R25.2; no longer C6.1, Q16.2, U$5.31
- net N$23: now also LED26.C, R26.2; no longer C1.1, Q16.1, U$5.30
- net N$24: now also LED27.C, R28.2; no longer R6.1, U$5.23
- net N$4: now also LED1.C, R14.2; no longer R5.2, R8.1, U$5.19
- net SCL: no longer U$5.9
- net SDA: no longer U$5.8
- net TORPEDO1_GATE: no longer U$5.11
- net TORPEDO2_GATE: no longer U$5.14
Routing:
- net +3V3: track 0.00 -> 267.3 mm, vias 1 -> 13
- net +24V: track 0.00 -> 128.0 mm, vias 0 -> 2
- net EXTRA1: track 0.00 -> 110.7 mm, vias 0 -> 5
- net +5V: track 0.00 -> 108.2 mm, vias 1 -> 4
- net AGND: track 0.00 -> 100.1 mm, vias 0 -> 28
- net SCL: track 0.00 -> 98.0 mm, vias 0 -> 6
- net SDA: track 0.00 -> 96.0 mm, vias 0 -> 6
- net EXTRA2: track 0.00 -> 90.8 mm, vias 0 -> 6
- net EXTRA3: track 0.00 -> 90.2 mm, vias 0 -> 6
- net EXTRA6: track 0.00 -> 89.7 mm, vias 0 -> 6
- net EXTRA5: track 0.00 -> 89.4 mm, vias 0 -> 6
- net EXTRA4: track 0.00 -> 79.5 mm, vias 0 -> 4
- net COIL_S_GATE: track 0.00 -> 79.4 mm, vias 0 -> 4
- net COIL_1_GATE: track 0.00 -> 76.6 mm, vias 0 -> 4
- net COIL_2_GATE: track 0.00 -> 72.4 mm, vias 0 -> 2
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- added copper zone on layer 1, net AGND
- added copper zone on layer 16, net AGND
- removed copper zone on layer 1, net GND
- removed copper zone on layer 16, net GND
Other:
- outline, holes or cut-outs redrawn

Commit message: Finished Actuator
Parts:
- removed J2: (no value), SparkFun-Connectors:1X04
- removed LED15, LED18: (no value), led:CHIPLED_0603
- removed R15: 220, resistor:R0805
- removed R16: 680, resistor:R0805
- added J3: (no value), SparkFun-Connectors:2X10
- moved LED25 41.0 mm to (12.7, 24.9)
- moved LED20 41.0 mm to (12.6, 38.3)
- moved LED21 41.0 mm to (12.6, 35.7)
- moved LED22 41.0 mm to (12.7, 33.0)
- moved LED23 41.0 mm to (12.7, 30.2)
- moved LED24 41.0 mm to (12.8, 27.5)
- moved LED26 41.0 mm to (12.7, 22.3)
- moved LED27 41.0 mm to (12.7, 19.7)
- moved R18 37.1 mm to (6.60, 40.4)
- moved R19 37.1 mm to (6.60, 37.0)
- moved R22 37.1 mm to (6.50, 33.5)
- moved R23 37.1 mm to (6.60, 30.0)
- moved R24 37.1 mm to (6.80, 26.3)
- moved R25 37.1 mm to (6.80, 22.6)
- moved R26 37.1 mm to (6.70, 19.1)
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Connections:
- removed net N$12: LED15.C, R15.2
- removed net N$13: LED18.C, R16.2
- removed net N$34: R27.1, S2.3, U2.7
- new net RESET: J3.15, R27.1, S2.3, U2.7
- net +12V: no longer LED18.A
- net +3V3: now also J3.1, J3.2; no longer J2.4
- net +5V: no longer LED15.A
- net AGND: now also J3.10, J3.12, J3.14, J3.16, J3.18, J3.20, J3.4, J3.6, J3.8; no longer J2.1, R15.1, R16.1
- net SWD_CLK: now also J3.9; no longer J2.2
- net SWD_IO: now also J3.7; no longer J2.3
Routing:
- net RESET: track 0.00 -> 62.8 mm, vias 0 -> 2
- net LED8: track 19.2 -> 65.4 mm, vias 0 -> 2
- net LED7: track 17.3 -> 62.4 mm, vias 0 -> 2
- net LED6: track 16.2 -> 59.4 mm, vias 0 -> 2
- net LED4: track 12.1 -> 54.0 mm, vias 0 -> 2
- net LED3: track 9.97 -> 51.7 mm, vias 0 -> 2
- net LED2: track 7.78 -> 49.5 mm, vias 0 -> 2
- net LED5: track 14.6 -> 56.1 mm, vias 0 -> 2
- net LED1: track 6.91 -> 47.8 mm, vias 0 -> 2
- net +3V3: track 267.3 -> 300.2 mm
- net USB_DN: track 47.3 -> 19.4 mm, vias 4 -> 2
- net N$34: track 25.4 -> 0.00 mm
- net SWD_CLK: track 19.8 -> 40.6 mm, vias 1 -> 3
- net SWD_IO: track 22.5 -> 42.6 mm, vias 1 -> 3
- net N$29: track 20.2 -> 11.0 mm, vias 2 -> 0
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Other:
- board text added: "Actuator"
- board text removed: "Board Name HERE!!!"

Commit message: Actuator Update
Parts:
- removed J3: (no value), SparkFun-Connectors:2X10
- removed LED19: (no value), led:CHIPLED_0603
- added DISCHARGING: (no value), led:CHIPLED_0603
- added SWDIO/SWDCLK/RESET: (no value), SparkFun-Connectors:2X10
- moved R17 5.97 mm to (22.8, 26.0)
- moved R21 3.00 mm to (28.0, 31.6)
- moved R30 0.30 mm to (31.8, 79.2)
- renumbered J1 to USB_ID/USB_DP/USB_DN, LED1 to CHARGING, LED20 to LIGHT1, LED21 to LIGHT2, LED22 to LIGHT3, LED23 to LIGHT4, LED24 to LIGHT5, LED25 to LIGHT6, LED26 to LIGHT7, LED27 to LIGHT8, P2 to ACTUATOR, S2 to RESET_SWITCH, U2 to MC
Connections:
- net +24V: now also DISCHARGING.A; no longer LED19.A
- net +3V3: now also SWDIO/SWDCLK/RESET.1, SWDIO/SWDCLK/RESET.2; no longer J3.1, J3.2
- net AGND: now also SWDIO/SWDCLK/RESET.10, SWDIO/SWDCLK/RESET.12, SWDIO/SWDCLK/RESET.14, SWDIO/SWDCLK/RESET.16, SWDIO/SWDCLK/RESET.18, SWDIO/SWDCLK/RESET.20, SWDIO/SWDCLK/RESET.4, SWDIO/SWDCLK/RESET.6, SWDIO/SWDCLK/RESET.8; no longer J3.10, J3.12, J3.14, J3.16, J3.18, J3.20, J3.4, J3.6, J3.8
- net N$15: now also DISCHARGING.C; no longer LED19.C
- net RESET: now also SWDIO/SWDCLK/RESET.15; no longer J3.15
- net SWD_CLK: now also SWDIO/SWDCLK/RESET.9; no longer J3.9
- net SWD_IO: now also SWDIO/SWDCLK/RESET.7; no longer J3.7
Routing:
- net RESET: track 62.8 -> 54.1 mm
- net AGND: track 91.5 -> 95.5 mm, vias 27 -> 28
- net +24V: track 128.0 -> 125.5 mm
- net N$26: track 25.4 -> 26.6 mm
- net +3V3: track 300.2 -> 301.4 mm
- net SWD_IO: track 42.6 -> 43.6 mm
- net SWD_CLK: track 40.6 -> 41.6 mm
Other:
- board text added: "Coils"
- board text added: "Dropper"
- board text added: "Torpedo"
- board text added: "U$3"

Commit message: Actuator Update
Connections:
- removed net MOBO_SWITCHED: ACTUATOR.12
Routing:
- net RESET: track 54.1 -> 63.4 mm
- net +5V: track 105.6 -> 104.2 mm
- net USB_DN: track 19.4 -> 18.9 mm
- net +24V: track 125.5 -> 126.1 mm
Changed lines of the file:
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@@
 Center for Automotive Research</text>
 <wire x1="62" y1="92.7" x2="68.5" y2="92.7" width="0.1524" layer="25"/>
-<text x="90.9" y="63.3" size="0.8128" layer="25" rot="R90">Coils</text>
-<wire x1="88.2" y1="52.1" x2="89.8" y2="52.1" width="0.1524" layer="25"/>
-<wire x1="89.8" y1="52.1" x2="89.8" y2="76.8" width="0.1524" layer="25"/>
-<wire x1="89.8" y1="76.8" x2="87.8" y2="76.8" width="0.1524" layer="25"/>
+<text x="85.2" y="62.1" size="0.8128" layer="25" rot="R90">Coils</text>
+<wire x1="88.2" y1="52.1" x2="85.7" y2="52.1" width="0.1524" layer="25"/>
+<wire x1="85.7" y1="52.1" x2="85.7" y2="76.8" width="0.1524" layer="25"/>
+<wire x1="85.7" y1="76.8" x2="87.8" y2="76.8" width="0.1524" layer="25"/>
 <wire x1="81.5" y1="60.3" x2="79.5" y2="60.3" width="0.1524" layer="25"/>
 <wire x1="79.5" y1="60.3" x2="79.5" y2="68.4" width="0.1524" layer="25"/>
@@
 <wire x1="44.5" y1="8.3" x2="44.5" y2="7.6" width="0.508" layer="1"/>
 <wire x1="96.1" y1="50.6" x2="96.1" y2="32.7" width="0.508" layer="1"/>
-<wire x1="44.5" y1="7.6" x2="44.5" y2="6.2" width="0.508" layer="1"/>
 </signal>
 <signal name="+3V3">
@@
 <wire x1="81.5" y1="53.3433" x2="82.0882" y2="53.9315" width="0.508" layer="1"/>
 <wire x1="19" y1="7.6" x2="16.75" y2="9.85" width="0.508" layer="1"/>
-<wire x1="16.75" y1="9.85" x2="16.6" y2="10" width="0.508" layer="1"/>
 <wire x1="10.6" y1="80.5" x2="12.8" y2="80.5" width="0.508" layer="1"/>
 <wire x1="12.8" y1="80.5" x2="21.3" y2="80.5" width="0.508" layer="1"/>
@@
 <wire x1="34.7556" y1="80.88523125" x2="35.02036875" y2="81.15" width="0.254" layer="1"/>
 <wire x1="35.02036875" y1="81.15" x2="35.77" y2="81.15" width="0.254" layer="1"/>
-<wire x1="35.77" y1="81.15" x2="35.75" y2="81.15" width="0.254" layer="1"/>
 <wire x1="21.6" y1="15.35" x2="22.95" y2="14" width="0.254" layer="1"/>
 <wire x1="22.95" y1="14" x2="27.2" y2="14" width="0.254" layer="1"/>
@@
 <contactref element="R26" pad="1"/>
 <contactref element="R28" pad="1"/>
-<wire x1="12.6" y1="93" x2="12.7" y2="92.9" width="0.1524" layer="1"/>
 <polygon width="0.1524" layer="16" thermals="no">
 <vertex x="1.9" y="8.9"/>
@@
 <wire x1="88.8" y1="52.7315" x2="87.6" y2="53.9315" width="0.508" layer="1"/>
 </signal>
-<signal name="MOBO_SWITCHED">
-<contactref element="ACTUATOR" pad="12"/>
-</signal>
 <signal name="COIL_5">
 <contactref element="ACTUATOR" pad="4"/>
@@
 <contactref element="Q17" pad="3"/>
 <contactref element="D8" pad="A"/>
-<wire x1="68.7225" y1="85.9775" x2="68.7" y2="86" width="0.1524" layer="1"/>
-<wire x1="68.7" y1="86" x2="73.2" y2="86" width="0.508" layer="1"/>
 <wire x1="73.2" y1="86" x2="75.1657" y2="86" width="0.6096" layer="1"/>
 <wire x1="75.1657" y1="86" x2="82.0882" y2="79.0775" width="0.6096" layer="1"/>
+<wire x1="73.2" y1="86" x2="68.7" y2="86" width="0.6096" layer="1"/>
 </signal>
 <signal name="DROPPER2">
@@
 <contactref element="Q12" pad="3"/>
 <contactref element="D9" pad="A"/>
-<wire x1="68.7135" y1="80.5865" x2="68.7" y2="80.6" width="0.1524" layer="1"/>
 <wire x1="68.7" y1="80.6" x2="73.2" y2="80.6" width="0.508" layer="1"/>
 <wire x1="73.2" y1="80.6" x2="73.3" y2="80.5" width="0.508" layer="1"/>
@@
 <wire x1="80.1" y1="40.5" x2="75.8" y2="40.5" width="1.27" layer="1"/>
 <wire x1="75.8" y1="40.5" x2="71.5" y2="40.5" width="1.27" layer="1"/>
-<wire x1="55.4" y1="64.25" x2="55.45" y2="64.3" width="0.1524" layer="1"/>
-<wire x1="55.45" y1="64.3" x2="57.8" y2="64.3" width="0.1524" layer="1"/>
 <wire x1="55.8" y1="72.75" x2="58.07" y2="72.75" width="0.1524" layer="1"/>
 <wire x1="58.07" y1="72.75" x2="58.6" y2="72.22" width="0.1524" layer="1"/>
@@
 <wire x1="33.176" y1="33.58" x2="28" y2="28.404" width="1.27" layer="1"/>
 <wire x1="28" y1="25.15" x2="28" y2="28.404" width="1.27" layer="1"/>
-<wire x1="58.3" y1="64.12" x2="57.8" y2="64.3" width="0" layer="19" extent="1-1"/>
+<wire x1="55.4" y1="64.25" x2="58.17" y2="64.25" width="0.1524" layer="1"/>
+<wire x1="58.17" y1="64.25" x2="58.3" y2="64.12" width="0.1524" layer="1"/>
 </signal>
 <signal name="ARM_TORPEDO">
@@
 <wire x1="70.55" y1="50.25" x2="70.5" y2="50.3" width="0.1524" layer="1"/>
 <via x="70.5" y="50.3" extent="1-16" drill="0.35"/>
-<wire x1="26.3" y1="71.68" x2="26.35" y2="71.73" width="0.1524" layer="1"/>
 <wire x1="65.5" y1="55.3" x2="64.8" y2="55.3" width="0.1524" layer="16"/>
 <via x="64.8" y="55.3" extent="1-16" drill="0.35"/>
@@
 <contactref element="Q17" pad="1"/>
 <contactref element="MC" pad="35"/>
-<wire x1="71.1" y1="86.95" x2="71.35" y2="86.7" width="0.1524" layer="1"/>
 <wire x1="71.1" y1="86.95" x2="69.35" y2="88.7" width="0.1524" layer="1"/>
 <via x="41.4" y="88.7" extent="1-16" drill="0.35"/>
@@
 <contactref element="R13" pad="2"/>
 <contactref element="MC" pad="44"/>
-<wire x1="19.5" y1="83.95" x2="19.9" y2="83.55" width="0.1524" layer="1"/>
 <wire x1="19.5" y1="83.95" x2="19.5" y2="82.5" width="0.1524" layer="1"/>
 <wire x1="19.5" y1="82.5" x2="19.7" y2="82.3" width="0.1524" layer="1"/>
@@
 <contactref element="MC" pad="20"/>
 <contactref element="LIGHT1" pad="A"/>
-<wire x1="13.35" y1="38.3" x2="13.45" y2="38.4" width="0.1524" layer="1"/>
 <wire x1="13.35" y1="38.3" x2="13.35" y2="66.75" width="0.1524" layer="1"/>
 <wire x1="13.35" y1="66.75" x2="13.5" y2="66.9" width="0.1524" layer="1"/>
@@
 <wire x1="15.2" y1="65.7" x2="15.2" y2="69.5" width="0.1524" layer="16"/>
 <via x="15.2" y="69.5" extent="1-16" drill="0.35"/>
-<wire x1="24.2986" y1="79.0186" x2="24.43" y2="79.15" width="0.1524" layer="1"/>
 <wire x1="15.2" y1="69.5" x2="15.2" y2="72.33105625" width="0.1524" layer="1"/>
-<wire x1="15.2" y1="72.33105625" x2="21.88754375" y2="79.0186" width="0.1524" layer="1"/>
-<wire x1="21.88754375" y1="79.0186" x2="24.2986" y2="79.0186" width="0.1524" layer="1"/>
+<wire x1="22.01894375" y1="79.15" x2="24.43" y2="79.15" width="0.1524" layer="1"/>
+<wire x1="15.2" y1="72.33105625" x2="22.01894375" y2="79.15" width="0.1524" layer="1"/>
 </signal>
 <signal name="LED3">
@@
 <wire x1="16.5" y1="73.2" x2="22" y2="78.7" width="0.1524" layer="1"/>
 <wire x1="22" y1="78.7" x2="24.38" y2="78.7" width="0.1524" layer="1"/>
-<wire x1="24.38" y1="78.7" x2="24.43" y2="78.65" width="0" layer="19" extent="1-1"/>
+<wire x1="24.38" y1="78.7" x2="24.43" y2="78.65" width="0.1524" layer="1"/>
 </signal>
 <signal name="LED4">
@@
 <via x="18" y="67" extent="1-16" drill="0.35"/>
 <wire x1="18" y1="67" x2="18" y2="74.2" width="0.1524" layer="1"/>
+<wire x1="18" y1="74.2" x2="21.95" y2="78.15" width="0.1524" layer="1"/>
 <wire x1="21.95" y1="78.15" x2="24.43" y2="78.15" width="0.1524" layer="1"/>
-<wire x1="18" y1="74.2" x2="21.95" y2="78.15" width="0.1524" layer="1"/>
 </signal>
 <signal name="LED5">
@@
 <contactref element="MC" pad="25"/>
 <contactref element="LIGHT6" pad="A"/>
-<wire x1="24.38" y1="77.2" x2="24.43" y2="77.15" width="0.1524" layer="1"/>
 <wire x1="13.45" y1="24.9" x2="21" y2="32.45" width="0.1524" layer="1"/>
 <wire x1="21" y1="32.45" x2="21" y2="59.4" width="0.1524" layer="1"/>
@@
 <contactref element="MC" pad="27"/>
 <contactref element="LIGHT8" pad="A"/>
-<wire x1="24.38" y1="76.2" x2="24.43" y2="76.15" width="0.1524" layer="1"/>
 <via x="24.3" y="56.1" extent="1-16" drill="0.35"/>
 <wire x1="17.7" y1="25.2" x2="21.2364" y2="28.7364" width="0.1524" layer="1"/>
@@
 <contactref element="RESET_SWITCH" pad="3"/>
 <contactref element="R27" pad="1"/>
-<wire x1="44.9394" y1="93.1488" x2="44.7882" y2="93.3" width="0.1524" layer="1"/>
 <via x="53.2" y="91.2" extent="1-16" drill="0.35"/>
 <wire x1="53.2" y1="91.2" x2="46.8882" y2="91.2" width="0.1524" layer="16"/>
 <wire x1="46.8882" y1="91.2" x2="44.9394" y2="93.1488" width="0.1524" layer="16"/>
-<wire x1="42.7" y1="95.3882" x2="42.7" y2="95.65" width="0.1524" layer="1"/>
-<wire x1="44.9394" y1="93.1488" x2="42.7" y2="95.3882" width="0.1524" layer="1"/>
 <wire x1="44.9394" y1="93.1488" x2="26.7488" y2="93.1488" width="0.1524" layer="1"/>
 <wire x1="26.7488" y1="93.1488" x2="25.3" y2="91.7" width="0.1524" layer="1"/>
@@
 <wire x1="25.3" y1="90.069275" x2="30.85" y2="84.519275" width="0.1524" layer="1"/>
 <wire x1="30.85" y1="84.519275" x2="30.85" y2="83.07" width="0.1524" layer="1"/>
-<wire x1="62.6" y1="91.3" x2="53.2" y2="91.2" width="0" layer="19" extent="1-1"/>
 <wire x1="71.48" y1="94.6" x2="68.18" y2="91.3" width="0.1524" layer="16"/>
 <wire x1="68.18" y1="91.3" x2="62.6" y2="91.3" width="0.1524" layer="16"/>
 <via x="62.6" y="91.3" extent="1-16" drill="0.35"/>
+<wire x1="53.2" y1="91.2" x2="53.3" y2="91.3" width="0.1524" layer="1"/>
+<wire x1="53.3" y1="91.3" x2="62.6" y2="91.3" width="0.1524" layer="1"/>
+<wire x1="42.7" y1="95.65" x2="42.7" y2="95.3882" width="0.1524" layer="1"/>
+<wire x1="42.7" y1="95.3882" x2="44.9394" y2="93.1488" width="0.1524" layer="1"/>
 </signal>
 </signals>
