File: Maelstrom Boards/Actuator/Actuator.sch (EAGLE design)
At the start: 65 parts, among them J1 USB_MINI-B_SMT, P2 39-30-16, Q1 MOSFET-NCH-AO3404A, Q12 MOSFET-NCH-AO3404A, Q13 MOSFET-NCH-AO3404A, Q14 MOSFET-NCH-AO3404A, Q15 MOSFET-NCH-AO3404A, Q17 MOSFET-NCH-AO3404A, Q18 FDD4141TO252, Q2 MOSFET-NCH-AO3404A, Q3 MOSFET-NCH-AO3404A, Q4 MOSFET-NCH-AO3404A, Q5 MOSFET-NCH-AO3404A, Q6 FDD4141TO252, U2 STM32F405RGT6, Y1 12MHz, Y3 32.768kHz

Commit message: Actuator new
Parts:
- removed C1, C6: 30pF, rcl:C-EUC0603
- removed C24: 220nF, rcl:C-EUC0603
- removed C25: 100nF, rcl:C-EUC0603
- removed Q16: (no value), crystal:CRYSTALHC49UP
- removed R42, R8: 10K, rcl:R-US_R0603
- removed R5: 100K, rcl:R-US_R0603
- removed R6: 5, rcl:R-US_R0603
- removed U$5: 18F4550, 18f4550:18F4550
- added LED1, LED15, LED18, LED19, LED20, LED21, LED22, LED23, LED24, LED25, LED26, LED27: (no value), led:LEDCHIPLED_0603
- added R14, R18, R19, R22, R23, R24, R25, R26, R28: 100, resistor:R-US_R0805
- added R15: 220, resistor:R-US_R0805
- added R16: 680, resistor:R-US_R0805
- added R17: 1.5k, resistor:R-US_R0805
Connections:
- removed net !MCLR!: U$5.!MCLR!/VPP
- removed net N$32: C24.1, U$5.VUSB
- removed net N$33: R42.1, U$5.RB5/PGM
- removed net PGC: U$5.RB6/PGC
- removed net PGD: U$5.RB7/PGD
- removed net PWM: U$5.PWM
- removed net USB+: U$5.USB+
- removed net USB-: U$5.USB-
- new net EXTRA1: U$1.SPARE2, U2.PC11
- new net EXTRA2: U$1.SPARE3, U2.PC12
- new net EXTRA3: U$1.SPARE4, U2.PD2
- new net EXTRA4: U$1.SPARE7, U2.PC10
- new net EXTRA5: U$1.SPARE6, U2.PB4
- new net EXTRA6: U$1.SPARE5, U2.PB3
- new net LED1: LED20.A, U2.PA4/USART2_CK
- new net LED2: LED21.A, U2.PA5/SPI1_SCK
- new net LED3: LED22.A, U2.PA6/SPI1_MISO
- new net LED4: LED23.A, U2.PA7/SPI1_MOSI
- new net LED5: LED24.A, U2.PC4
- new net LED6: LED25.A, U2.PC5
- new net LED7: LED26.A, U2.PB0
- new net LED8: LED27.A, U2.PB1
- new net N$12: LED15.C, R15.2
- new net N$13: LED18.C, R16.2
- new net N$16: LED20.C, R18.2
- new net N$17: LED21.C, R19.2
- new net N$18: LED22.C, R22.2
- new net N$19: LED23.C, R23.2
- new net N$21: LED24.C, R24.2
- new net SMBA: U2.PB5
- new net SWD_CLK: J2.2, U2.PA14/JTCK-SWCLK
- new net SWD_IO: J2.3, U2.PA13/JMS-SWDIO
- net +12V: now also LED18.A
- net +24V: now also LED19.A; no longer R5.1
- net +3V3: now also J2.4, LED1.A; no longer C25.1, U$5.VDD
- net +5V: now also LED15.A
- net AGND: now also J2.1, R14.1, R15.1, R16.1, R17.1, R18.1, R19.1, R22.1, R23.1, R24.1, R25.1, R26.1, R28.1; no longer C1.2, C24.2, C25.2, C6.2, R42.2, R8.2, U$5.VSS
- net ARM_TORPEDO: no longer U$5.B2
- net COIL_1_GATE: no longer U$5.D0
- net COIL_2_GATE: no longer U$5.D1
- net COIL_3_GATE: no longer U$5.D2
- net COIL_4_GATE: no longer U$5.D3
- net COIL_5_GATE: no longer U$5.D4
- net COIL_S_GATE: no longer U$5.D5
- net DROPPER1_GATE: no longer U$5.D6
- net DROPPER2_GATE: no longer U$5.D7
- net N$15: now also LED19.C, R17.2; no longer R6.2
- net N$22: now also LED25.C, R25.2; no longer C6.1, Q16.2, U$5.OSC2
- net N$23: now also LED26.C, R26.2; no longer C1.1, Q16.1, U$5.OSC1
- net N$24: now also LED27.C, R28.2; no longer R6.1, U$5.RUN
- net N$4: now also LED1.C, R14.2; no longer R5.2, R8.1, U$5.A0
- net SCL: no longer U$5.SCL
- net SDA: no longer U$5.SDA
- net TORPEDO1_GATE: no longer U$5.B3
- net TORPEDO2_GATE: no longer U$5.B4
Other:
- moved on the sheet: C4, C5, D10, D8, Q17, R20, R21

Commit message: Finished Actuator
Parts:
- removed J2: (no value), SparkFun-Connectors:CONN_04
- removed LED15, LED18: (no value), led:LEDCHIPLED_0603
- removed R15: 220, resistor:R-US_R0805
- removed R16: 680, resistor:R-US_R0805
- added J3: (no value), SparkFun-Connectors:CONN_10X2
Connections:
- removed net N$12: LED15.C, R15.2
- removed net N$13: LED18.C, R16.2
- removed net N$34: R27.1, S2.2, U2.NRST
- new net RESET: J3.15, R27.1, S2.2, U2.NRST
- net +12V: no longer LED18.A
- net +3V3: now also J3.1, J3.2; no longer J2.4
- net +5V: no longer LED15.A
- net AGND: now also J3.10, J3.12, J3.14, J3.16, J3.18, J3.20, J3.4, J3.6, J3.8; no longer J2.1, R15.1, R16.1
- net SWD_CLK: now also J3.9; no longer J2.2
- net SWD_IO: now also J3.7; no longer J2.3

Commit message: Actuator Update
Parts:
- renumbered J1 to USB_ID/USB_DP/USB_DN, J3 to SWDIO/SWDCLK/RESET, LED1 to CHARGING, LED19 to DISCHARGING, LED20 to LIGHT1, LED21 to LIGHT2, LED22 to LIGHT3, LED23 to LIGHT4, LED24 to LIGHT5, LED25 to LIGHT6, LED26 to LIGHT7, LED27 to LIGHT8, P2 to ACTUATOR, S2 to RESET_SWITCH, U2 to MC

Commit message: Actuator Update
Connections:
- removed net MOBO_SWITCHED: ACTUATOR.12
Changed lines of the file:
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@@
-</segment>
-</net>
-<net name="MOBO_SWITCHED" class="0">
-<segment>
-<wire x1="271.78" y1="144.78" x2="271.78" y2="147.32" width="0.1524" layer="91"/>
-<wire x1="271.78" y1="147.32" x2="274.32" y2="147.32" width="0.1524" layer="91"/>
-<label x="274.32" y="147.32" size="1.778" layer="95" xref="yes"/>
-<pinref part="ACTUATOR" gate="G$1" pin="12"/>
-<wire x1="271.78" y1="144.78" x2="259.08" y2="144.78" width="0.1524" layer="91"/>
 </segment>
 </net>
