File: Eddy Boards/Backplane/Eddy Backplane.sch (EAGLE design)
At the start: 46 parts, among them J1 USB_MINI-B_SMT, P1 39-30-02_S, P3 39-30-04_S

Commit message: backplane update
Other:
- moved on the sheet: 16MHZ, 32.768KHZ, C11, C12, C8, C9
