File: Titan Boards/Battery Balancer/Titan_Balancer.brd (EAGLE design)
At the start: 101.6 x 101.6 mm, 83 parts, among them IC1 REG1117, IC2 SN74LV11AD, P1 39-30-04?, P2 39-30-10?, P4 39-30-04?, P5 39-30-06?, Q1 SPD30P06PTO252, Q12 310mA/60V/1.6Ω, Q2 SPB80P06P, Q3 SPB80P06P, Q4 SPD30P06PTO252, U1 I6A4W020A033V-001-R, U2 I6A4W020A033V-001-R

Commit message: put led's to and gate, voltage needs stepped up or down
Connections:
- new net N$31: 5V.C
- net 12V_LED: now also 12V.A, IC2.9
- net 3V3_LED: now also 3V3.A, IC2.1, IC2.2
- net 5V_LED: now also 5V.A, IC2.13
- net BALANCED_LED: now also BALANCED.A, BALANCED.C, IC2.10, IC2.11
- net N$20: now also 3V3.C; no longer 5V.A
- net N$26: now also IC2.8; no longer BALANCED.A
- net N$27: now also IC2.6; no longer STBD.A
- net N$28: now also PORT.C; no longer PORT.A
- net N$29: now also STBD.C; no longer 3V3.A
- net N$30: now also 12V.C; no longer IC2.11, IC2.12
- net N$9: now also IC2.12; no longer 12V.A
- net PORT_LED: now also IC2.3, IC2.4, PORT.A
- net STBD_LED: now also IC2.5, STBD.A
Changed lines of the file:
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@@
 <?xml version="1.0" encoding="utf-8"?>
 <!DOCTYPE eagle SYSTEM "eagle.dtd">
-<eagle version="9.5.2">
+<eagle version="9.6.2">
 <drawing>
 <settings>
@@
 <contactref element="R12" pad="2"/>
 <contactref element="R13" pad="2"/>
+<contactref element="IC2" pad="5"/>
+<contactref element="STBD" pad="A"/>
+<wire x1="-5.754" y1="-48.26" x2="-69.26" y2="-182.626" width="0" layer="19" extent="1-1"/>
 <wire x1="-5.754" y1="-40.386" x2="-5.754" y2="-48.26" width="0" layer="19" extent="1-1"/>
+<wire x1="157.214" y1="47.752" x2="-5.754" y2="-40.386" width="0" layer="19" extent="1-1"/>
 </signal>
 <signal name="PORT_LED">
 <contactref element="R15" pad="2"/>
 <contactref element="R18" pad="2"/>
+<contactref element="IC2" pad="3"/>
+<contactref element="IC2" pad="4"/>
+<contactref element="PORT" pad="A"/>
+<wire x1="-69.26" y1="-180.086" x2="-69.26" y2="-181.356" width="0" layer="19" extent="1-1"/>
+<wire x1="2.12" y1="-18.542" x2="-69.26" y2="-180.086" width="0" layer="19" extent="1-1"/>
 <wire x1="2.374" y1="-12.446" x2="2.12" y2="-18.542" width="0" layer="19" extent="1-1"/>
+<wire x1="166.104" y1="65.278" x2="2.374" y2="-12.446" width="0" layer="19" extent="1-1"/>
 </signal>
 <signal name="BALANCED_LED">
 <contactref element="R19" pad="1"/>
 <contactref element="R14" pad="1"/>
+<contactref element="IC2" pad="11"/>
+<contactref element="IC2" pad="10"/>
+<contactref element="BALANCED" pad="A"/>
+<contactref element="BALANCED" pad="C"/>
+<wire x1="-63.836" y1="-182.626" x2="-63.836" y2="-181.356" width="0" layer="19" extent="1-1"/>
+<wire x1="5.908" y1="-26.162" x2="-63.836" y2="-181.356" width="0" layer="19" extent="1-1"/>
 <wire x1="5.754" y1="-20.32" x2="5.908" y2="-26.162" width="0" layer="19" extent="1-1"/>
+<wire x1="171.208" y1="72.898" x2="5.754" y2="-20.32" width="0" layer="19" extent="1-1"/>
+<wire x1="172.708" y1="72.898" x2="171.208" y2="72.898" width="0" layer="19" extent="1-1"/>
 </signal>
 <signal name="3V3_LED">
 <contactref element="R11" pad="1"/>
+<contactref element="IC2" pad="1"/>
+<contactref element="IC2" pad="2"/>
+<contactref element="3V3" pad="A"/>
+<wire x1="-69.26" y1="-177.546" x2="-69.26" y2="-178.816" width="0" layer="19" extent="1-1"/>
+<wire x1="2.198" y1="-156.718" x2="-69.26" y2="-177.546" width="0" layer="19" extent="1-1"/>
+<wire x1="169.152" y1="51.308" x2="2.198" y2="-156.718" width="0" layer="19" extent="1-1"/>
 </signal>
 <signal name="N$8">
@@
 <signal name="12V_LED">
 <contactref element="R16" pad="1"/>
+<contactref element="IC2" pad="9"/>
+<contactref element="12V" pad="A"/>
+<wire x1="168.822" y1="36.83" x2="-63.836" y2="-183.896" width="0" layer="19" extent="1-1"/>
+<wire x1="172.986" y1="38.354" x2="168.822" y2="36.83" width="0" layer="19" extent="1-16"/>
 </signal>
 <signal name="N$22">
@@
 <signal name="5V_LED">
 <contactref element="R17" pad="1"/>
+<contactref element="IC2" pad="13"/>
+<contactref element="5V" pad="A"/>
+<wire x1="163.742" y1="43.18" x2="-63.836" y2="-178.816" width="0" layer="19" extent="1-1"/>
+<wire x1="168.922" y1="45.212" x2="163.742" y2="43.18" width="0" layer="19" extent="1-16"/>
 </signal>
 <signal name="N$10">
@@
 </signal>
 <signal name="N$9">
-<contactref element="12V" pad="A"/>
-</signal>
-<signal name="N$20">
-<contactref element="5V" pad="A"/>
+<contactref element="IC2" pad="12"/>
 </signal>
 <signal name="N$26">
-<contactref element="BALANCED" pad="A"/>
+<contactref element="IC2" pad="8"/>
 </signal>
 <signal name="N$27">
-<contactref element="STBD" pad="A"/>
+<contactref element="IC2" pad="6"/>
+</signal>
+<signal name="N$20">
+<contactref element="3V3" pad="C"/>
 </signal>
 <signal name="N$28">
-<contactref element="PORT" pad="A"/>
+<contactref element="PORT" pad="C"/>
 </signal>
 <signal name="N$29">
-<contactref element="3V3" pad="A"/>
+<contactref element="STBD" pad="C"/>
 </signal>
 <signal name="N$30">
-<contactref element="IC2" pad="12"/>
-<contactref element="IC2" pad="11"/>
-<wire x1="-63.836" y1="-180.086" x2="-63.836" y2="-181.356" width="0" layer="19" extent="1-1"/>
+<contactref element="12V" pad="C"/>
+</signal>
+<signal name="N$31">
+<contactref element="5V" pad="C"/>
 </signal>
 </signals>
