File: Titan Boards/Copro/CoPro.brd (EAGLE design)
At the start: 101.6 x 101.6 mm, 91 parts, among them P2 RB1-125BAG1A, Q1 310mA/60V/1.6Ω, Q10 310mA/60V/1.6Ω, Q2 310mA/60V/1.6Ω, Q3 310mA/60V/1.6Ω, Q4 310mA/60V/1.6Ω, Q5 310mA/60V/1.6Ω, Q6 310mA/60V/1.6Ω, Q7 310mA/60V/1.6Ω, Q8 310mA/60V/1.6Ω, Q9 310mA/60V/1.6Ω, U1 SN74LVC3G04DCUT, U2 SN74LVC1G11DCKR, Y1 25Mhz, Y2 12MHz, Y3 32.768kHz

Commit message: Changed Oscillator from 12Hz to 16Hz
Parts:
- Y2: value 12MHz -> 16MHz
Changed lines of the file:
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@@
 <attribute name="VALUE" x="53.04956875" y="59.39355" size="2.002690625" layer="27" rot="R180" align="top-left"/>
 </element>
-<element name="Y2" library="SparkFun-Clocks" library_urn="urn:adsk.eagle:library:511" package="HC49US" package3d_urn="urn:adsk.eagle:package:37515/1" value="12MHz" x="58.166" y="50.292" smashed="yes" rot="R270">
+<element name="Y2" library="SparkFun-Clocks" library_urn="urn:adsk.eagle:library:511" package="HC49US" package3d_urn="urn:adsk.eagle:package:37515/1" value="16MHz" x="58.166" y="50.292" smashed="yes" rot="R270">
 <attribute name="NAME" x="60.706" y="50.292" size="0.6096" layer="25" font="vector" ratio="20" rot="R270" align="bottom-center"/>
 <attribute name="PROD_ID" value="XTAL-08181" x="78.74" y="82.55" size="1.778" layer="27" rot="R270" display="off"/>
