File: Titan Boards/ESC/ESC.sch (EAGLE design)
At the start: 113 parts, among them Q1 2N2222, Q10 BSS138, Q3 BSS138, Q4 BSS138, Q5 BSS138, Q6 BSS138, Q7 BSS138, Q8 BSS138, Q9 BSS138

Commit message: more esc work
Connections:
- removed net N$1 (its old number): 24-PIN_CONNECTOR.7,WHITE, 3-PIN_1.WHITE
- removed net N$13: 24-PIN_CONNECTOR.8,WHITE, 3-PIN_5.WHITE
- removed net N$14: 24-PIN_CONNECTOR.8,GREEN, 3-PIN_5.GREEN
- removed net N$15: 24-PIN_CONNECTOR.8,BLUE, 3-PIN_5.BLUE
- removed net N$16: 24-PIN_CONNECTOR.6,WHITE, 3-PIN_6.WHITE
- removed net N$17: 24-PIN_CONNECTOR.6,GREEN, 3-PIN_6.GREEN
- removed net N$18: 24-PIN_CONNECTOR.6,BLUE, 3-PIN_6.BLUE
- removed net N$19: 24-PIN_CONNECTOR.4,WHITE, 3-PIN_7.WHITE
- removed net N$2 (its old number): 24-PIN_CONNECTOR.7,GREEN, 3-PIN_1.GREEN
- removed net N$20: 24-PIN_CONNECTOR.4,BLUE, 3-PIN_7.BLUE
- removed net N$21: 24-PIN_CONNECTOR.4,GREEN, 3-PIN_7.GREEN
- removed net N$22: 24-PIN_CONNECTOR.2,BLUE, 3-PIN_8.BLUE
- removed net N$23: 24-PIN_CONNECTOR.2,GREEN, 3-PIN_8.GREEN
- removed net N$24: 24-PIN_CONNECTOR.2,WHITE, 3-PIN_8.WHITE
- removed net N$3 (its old number): 24-PIN_CONNECTOR.7,BLUE, 3-PIN_1.BLUE
- removed net N$4 (its old number): 24-PIN_CONNECTOR.5,WHITE, 3-PIN_2.WHITE
- removed net N$5 (its old number): 24-PIN_CONNECTOR.5,GREEN, 3-PIN_2.GREEN
- removed net N$6 (its old number): 24-PIN_CONNECTOR.5,BLUE, 3-PIN_2.BLUE

Commit message: Titan ESC updates
Connections:
- new net N$10: 24-PIN_CONNECTOR.7,BLUE, 3-PIN_1.BLUE
- new net N$11: 24-PIN_CONNECTOR.7,GREEN, 3-PIN_1.GREEN
- new net N$12: 24-PIN_CONNECTOR.7,WHITE, 3-PIN_1.WHITE
- new net N$13: 24-PIN_CONNECTOR.8,BLUE, 3-PIN_5.WHITE
- new net N$14: 24-PIN_CONNECTOR.8,GREEN, 3-PIN_5.GREEN
- new net N$15: 24-PIN_CONNECTOR.8,WHITE, 3-PIN_5.BLUE
- new net N$16: 24-PIN_CONNECTOR.6,WHITE, 3-PIN_6.WHITE
- new net N$17: 24-PIN_CONNECTOR.6,GREEN, 3-PIN_6.GREEN
- new net N$18: 24-PIN_CONNECTOR.6,BLUE, 3-PIN_6.BLUE
- new net N$19: 24-PIN_CONNECTOR.4,BLUE, 3-PIN_7.BLUE
- new net N$20: 24-PIN_CONNECTOR.4,GREEN, 3-PIN_7.GREEN
- new net N$21: 24-PIN_CONNECTOR.4,WHITE, 3-PIN_7.WHITE
- new net N$22: 24-PIN_CONNECTOR.2,BLUE, 3-PIN_8.BLUE
- new net N$23: 24-PIN_CONNECTOR.2,GREEN, 3-PIN_8.GREEN
- new net N$24: 24-PIN_CONNECTOR.2,WHITE, 3-PIN_8.WHITE
- new net N$7: 24-PIN_CONNECTOR.5,BLUE, 3-PIN_2.BLUE
- new net N$8: 24-PIN_CONNECTOR.5,GREEN, 3-PIN_2.GREEN
- new net N$9: 24-PIN_CONNECTOR.5,WHITE, 3-PIN_2.WHITE
Other:
- note added: "Worthy of more consideration"
- note added: "failed more consideration"
- note added: "worthy of re-evaluation"
Changed lines of the file:
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@@
 <text x="12.7" y="205.74" size="1.778" layer="150">Top Side Devices</text>
 <text x="144.78" y="172.72" size="1.778" layer="150">Bottom Side Devices</text>
+<text x="340.36" y="180.34" size="1.778" layer="91">Worthy of more consideration</text>
+<text x="340.36" y="177.8" size="1.778" layer="91">failed more consideration</text>
+<text x="340.36" y="175.26" size="1.778" layer="91">worthy of re-evaluation</text>
 </plain>
 <instances>
@@
 </instance>
 <instance part="24-PIN_CONNECTOR" gate="G$1" x="154.94" y="231.14" smashed="yes" rot="R90"/>
-<instance part="3-PIN_5" gate="G$1" x="76.2" y="203.2" smashed="yes" rot="R270"/>
-<instance part="3-PIN_1" gate="G$1" x="91.44" y="180.34" smashed="yes" rot="R270"/>
-<instance part="3-PIN_2" gate="G$1" x="121.92" y="180.34" smashed="yes" rot="R270"/>
-<instance part="3-PIN_7" gate="G$1" x="45.72" y="203.2" smashed="yes" rot="R270"/>
-<instance part="3-PIN_6" gate="G$1" x="60.96" y="180.34" smashed="yes" rot="R270"/>
+<instance part="3-PIN_5" gate="G$1" x="22.86" y="198.12" smashed="yes" rot="R180"/>
+<instance part="3-PIN_1" gate="G$1" x="45.72" y="203.2" smashed="yes" rot="R270"/>
+<instance part="3-PIN_2" gate="G$1" x="76.2" y="203.2" smashed="yes" rot="R270"/>
+<instance part="3-PIN_7" gate="G$1" x="116.84" y="177.8" smashed="yes"/>
+<instance part="3-PIN_6" gate="G$1" x="55.88" y="198.12" smashed="yes" rot="R180"/>
 <instance part="3-PIN_3" gate="G$1" x="106.68" y="203.2" smashed="yes" rot="R270"/>
 <instance part="3-PIN_4" gate="G$1" x="137.16" y="203.2" smashed="yes" rot="R270"/>
-<instance part="3-PIN_8" gate="G$1" x="25.4" y="180.34" smashed="yes" rot="R270"/>
+<instance part="3-PIN_8" gate="G$1" x="152.4" y="180.34" smashed="yes"/>
 <instance part="POWER_INPUT" gate="G$1" x="200.66" y="195.58" smashed="yes"/>
 <instance part="GND2" gate="1" x="218.44" y="185.42" smashed="yes">
@@
 <pinref part="THRUSTER_PWM_1" gate="A" pin="3"/>
 <wire x1="271.78" y1="231.14" x2="264.16" y2="231.14" width="0.1524" layer="91"/>
+<pinref part="THRUSTER_PWM_2" gate="A" pin="3"/>
 <wire x1="264.16" y1="231.14" x2="264.16" y2="215.9" width="0.1524" layer="91"/>
-<pinref part="THRUSTER_PWM_2" gate="A" pin="3"/>
 <wire x1="264.16" y1="215.9" x2="271.78" y2="215.9" width="0.1524" layer="91"/>
 <pinref part="THRUSTER_PWM_3" gate="A" pin="3"/>
@@
 </segment>
 </net>
+<net name="N$7" class="0">
+<segment>
+<pinref part="24-PIN_CONNECTOR" gate="G$1" pin="5,BLUE"/>
+<pinref part="3-PIN_2" gate="G$1" pin="BLUE"/>
+<wire x1="91.44" y1="215.9" x2="91.44" y2="226.06" width="0.1524" layer="91"/>
+</segment>
+</net>
+<net name="N$8" class="0">
+<segment>
+<pinref part="24-PIN_CONNECTOR" gate="G$1" pin="5,GREEN"/>
+<pinref part="3-PIN_2" gate="G$1" pin="GREEN"/>
+<wire x1="86.36" y1="215.9" x2="86.36" y2="226.06" width="0.1524" layer="91"/>
+</segment>
+</net>
+<net name="N$9" class="0">
+<segment>
+<pinref part="24-PIN_CONNECTOR" gate="G$1" pin="5,WHITE"/>
+<pinref part="3-PIN_2" gate="G$1" pin="WHITE"/>
+<wire x1="81.28" y1="215.9" x2="81.28" y2="226.06" width="0.1524" layer="91"/>
+</segment>
+</net>
+<net name="N$10" class="0">
+<segment>
+<pinref part="24-PIN_CONNECTOR" gate="G$1" pin="7,BLUE"/>
+<pinref part="3-PIN_1" gate="G$1" pin="BLUE"/>
+<wire x1="60.96" y1="215.9" x2="60.96" y2="226.06" width="0.1524" layer="91"/>
+</segment>
+</net>
+<net name="N$11" class="0">
+<segment>
+<pinref part="24-PIN_CONNECTOR" gate="G$1" pin="7,GREEN"/>
+<pinref part="3-PIN_1" gate="G$1" pin="GREEN"/>
+<wire x1="55.88" y1="215.9" x2="55.88" y2="226.06" width="0.1524" layer="91"/>
+</segment>
+</net>
+<net name="N$12" class="0">
+<segment>
+<pinref part="24-PIN_CONNECTOR" gate="G$1" pin="7,WHITE"/>
+<pinref part="3-PIN_1" gate="G$1" pin="WHITE"/>
+<wire x1="50.8" y1="215.9" x2="50.8" y2="226.06" width="0.1524" layer="91"/>
+</segment>
+</net>
+<net name="N$14" class="0">
+<segment>
+<pinref part="3-PIN_5" gate="G$1" pin="GREEN"/>
+<wire x1="40.64" y1="226.06" x2="40.64" y2="187.96" width="0.1524" layer="91"/>
+<wire x1="40.64" y1="187.96" x2="35.56" y2="187.96" width="0.1524" layer="91"/>
+<pinref part="24-PIN_CONNECTOR" gate="G$1" pin="8,GREEN"/>
+</segment>
+</net>
+<net name="N$16" class="0">
+<segment>
+<pinref part="24-PIN_CONNECTOR" gate="G$1" pin="6,WHITE"/>
+<pinref part="3-PIN_6" gate="G$1" pin="WHITE"/>
+<wire x1="76.2" y1="226.06" x2="76.2" y2="193.04" width="0.1524" layer="91"/>
+<wire x1="76.2" y1="193.04" x2="68.58" y2="193.04" width="0.1524" layer="91"/>
+</segment>
+</net>
+<net name="N$17" class="0">
+<segment>
+<pinref part="24-PIN_CONNECTOR" gate="G$1" pin="6,GREEN"/>
+<pinref part="3-PIN_6" gate="G$1" pin="GREEN"/>
+<wire x1="71.12" y1="226.06" x2="71.12" y2="187.96" width="0.1524" layer="91"/>
+<wire x1="71.12" y1="187.96" x2="68.58" y2="187.96" width="0.1524" layer="91"/>
+</segment>
+</net>
+<net name="N$18" class="0">
+<segment>
+<pinref part="24-PIN_CONNECTOR" gate="G$1" pin="6,BLUE"/>
+<pinref part="3-PIN_6" gate="G$1" pin="BLUE"/>
+<wire x1="66.04" y1="226.06" x2="66.04" y2="182.88" width="0.1524" layer="91"/>
+<wire x1="66.04" y1="182.88" x2="68.58" y2="182.88" width="0.1524" layer="91"/>
+</segment>
+</net>
+<net name="N$13" class="0">
+<segment>
+<pinref part="24-PIN_CONNECTOR" gate="G$1" pin="8,BLUE"/>
+<pinref part="3-PIN_5" gate="G$1" pin="WHITE"/>
+<wire x1="35.56" y1="226.06" x2="35.56" y2="193.04" width="0.1524" layer="91"/>
+</segment>
+</net>
+<net name="N$15" class="0">
+<segment>
+<pinref part="3-PIN_5" gate="G$1" pin="BLUE"/>
+<wire x1="35.56" y1="182.88" x2="45.72" y2="182.88" width="0.1524" layer="91"/>
+<pinref part="24-PIN_CONNECTOR" gate="G$1" pin="8,WHITE"/>
+<wire x1="45.72" y1="182.88" x2="45.72" y2="226.06" width="0.1524" layer="91"/>
+</segment>
+</net>
+<net name="N$19" class="0">
+<segment>
+<pinref part="24-PIN_CONNECTOR" gate="G$1" pin="4,BLUE"/>
+<pinref part="3-PIN_7" gate="G$1" pin="BLUE"/>
+<wire x1="96.52" y1="226.06" x2="96.52" y2="193.04" width="0.1524" layer="91"/>
+<wire x1="96.52" y1="193.04" x2="104.14" y2="193.04" width="0.1524" layer="91"/>
+</segment>
+</net>
+<net name="N$20" class="0">
+<segment>
+<pinref part="24-PIN_CONNECTOR" gate="G$1" pin="4,GREEN"/>
+<pinref part="3-PIN_7" gate="G$1" pin="GREEN"/>
+<wire x1="101.6" y1="226.06" x2="101.6" y2="187.96" width="0.1524" layer="91"/>
+<wire x1="101.6" y1="187.96" x2="104.14" y2="187.96" width="0.1524" layer="91"/>
+</segment>
+</net>
+<net name="N$21" class="0">
+<segment>
+<pinref part="24-PIN_CONNECTOR" gate="G$1" pin="4,WHITE"/>
+<pinref part="3-PIN_7" gate="G$1" pin="WHITE"/>
+<wire x1="106.68" y1="226.06" x2="106.68" y2="182.88" width="0.1524" layer="91"/>
+<wire x1="106.68" y1="182.88" x2="104.14" y2="182.88" width="0.1524" layer="91"/>
+</segment>
+</net>
+<net name="N$22" class="0">
+<segment>
+<pinref part="24-PIN_CONNECTOR" gate="G$1" pin="2,BLUE"/>
+<pinref part="3-PIN_8" gate="G$1" pin="BLUE"/>
+<wire x1="127" y1="226.06" x2="127" y2="195.58" width="0.1524" layer="91"/>
+<wire x1="127" y1="195.58" x2="139.7" y2="195.58" width="0.1524" layer="91"/>
+</segment>
+</net>
+<net name="N$23" class="0">
+<segment>
+<pinref part="24-PIN_CONNECTOR" gate="G$1" pin="2,GREEN"/>
+<pinref part="3-PIN_8" gate="G$1" pin="GREEN"/>
+<wire x1="132.08" y1="226.06" x2="132.08" y2="190.5" width="0.1524" layer="91"/>
+<wire x1="132.08" y1="190.5" x2="139.7" y2="190.5" width="0.1524" layer="91"/>
+</segment>
+</net>
+<net name="N$24" class="0">
+<segment>
+<pinref part="24-PIN_CONNECTOR" gate="G$1" pin="2,WHITE"/>
+<pinref part="3-PIN_8" gate="G$1" pin="WHITE"/>
+<wire x1="137.16" y1="226.06" x2="137.16" y2="185.42" width="0.1524" layer="91"/>
+<wire x1="137.16" y1="185.42" x2="139.7" y2="185.42" width="0.1524" layer="91"/>
+</segment>
+</net>

Commit message: more changes to ESC board
Parts:
- removed Q10, Q9: BSS138, SparkFun-DiscreteSemi:MOSFET-NCH-BSS138
- removed R29, R30, R31, R32, R33, R34, R35, R36: 2k, rcl:R-US_R0603
- removed R37: 4.7K, rcl:R-US_R0603
- added IC1: 7425D, 74xx-us:7425D
- added IC2: 74AHC1G08DBV, 74xx-little-us:74AHC1G08DBV
- added Q2: 5.8A/30V/35mΩ, SparkFun-DiscreteSemi:MOSFET-NCH-AO3404A
- D10, D3, D4, D5, D6, D7, D8, D9: value RED -> Red
- Q1: value 2N2222 -> 5.8A/30V/35mΩ; device SparkFun-DiscreteSemi:TRANS_NPN-MMBT2222AL -> SparkFun-DiscreteSemi:MOSFET-NCH-AO3404A
- Q3, Q4, Q5, Q6, Q7, Q8: value BSS138 -> 5.8A/30V/35mΩ; device SparkFun-DiscreteSemi:MOSFET-NCH-BSS138 -> SparkFun-DiscreteSemi:MOSFET-NCH-AO3404A
- R10, R13, R16, R4, R7: value 190 -> (none)
- R11, R14, R17, R2, R20, R23, R5, R8: value 128 -> (none)
- R12, R15, R18, R6, R9: value 2.2K -> 28
- R19, R22, R25: value 190 -> 28
- R21, R24, R3: value 2.2K -> (none)
Connections:
- removed net N$54: D10.A, R23.1
- removed net N$59: D2.C, R28.1
- new net N$32: D3.C, Q1.D
- new net NOR_1_OUT: IC1A.O, IC2A.I0
- new net NOR_2_OUT: IC1B.O, IC2A.I1
- net +5V: now also IC1A.G, IC1B.G, IC1P.VCC, IC2P.VCC, R12.2, R15.2, R18.2, R19.2, R22.2, R25.2, R6.2, R9.2; no longer Q1.C, R11.2, R14.2, R17.2, R2.2, R20.2, R23.2, R5.2, R8.2
- net FAULT_1: now also IC1A.I0, Q1.G, R2.1, R3.2; no longer D3.C, Q3.D, R33.1
- net FAULT_2: now also IC1A.I1, Q2.G, R4.1, R5.2; no longer D4.C, Q4.D, R32.1
- net FAULT_3: now also IC1A.I2, Q3.G, R7.1, R8.2; no longer D5.C, Q5.D, R31.1
- net FAULT_4: now also IC1A.I3, Q4.G, R10.1, R11.2; no longer D6.C, Q6.D, R30.1
- net FAULT_5: now also IC1B.I0, Q5.G, R13.1, R14.2; no longer D7.C, Q7.D, R29.1
- net FAULT_6: now also IC1B.I1, Q6.G, R16.1, R17.2; no longer D8.C, Q8.D, R34.1
- net FAULT_7: now also IC1B.I2, Q7.G, R20.1, R21.2; no longer D9.C, Q9.D, R35.1
- net FAULT_8: now also IC1B.I3, Q8.G, R23.1, R24.2; no longer D10.C, Q10.D, R36.1
- net FUSE_1_TRIGGER: now also R2.2; no longer R3.2
- net FUSE_2_TRIGGER: now also R4.2; no longer R6.2
- net FUSE_3_TRIGGER: now also R7.2; no longer R9.2
- net FUSE_4_TRIGGER: now also R10.2; no longer R12.2
- net FUSE_5_TRIGGER: now also R13.2; no longer R15.2
- net FUSE_6_TRIGGER: now also R16.2; no longer R18.2
- net FUSE_7_TRIGGER: now also R20.2; no longer R21.2
- net FUSE_8_TRIGGER: now also R23.2; no longer R24.2
- net GND: now also D2.C, IC1P.GND, IC2P.GND, Q1.S, Q2.S, R11.1, R14.1, R17.1, R21.1, R24.1, R3.1, R5.1, R8.1; no longer Q10.S, Q9.S, R10.1, R13.1, R16.1, R19.1, R22.1, R25.1, R28.2, R37.2, R4.1, R7.1
- net N$13: now also 24-PIN_CONNECTOR.8,WHITE; no longer 24-PIN_CONNECTOR.8,BLUE
- net N$15: now also 24-PIN_CONNECTOR.8,BLUE; no longer 24-PIN_CONNECTOR.8,WHITE
- net N$31: now also IC2A.O, R28.2; no longer D3.A, R2.1
- net N$33: now also D3.A, R18.1; no longer D4.A, R5.1
- net N$34: now also D4.C, Q2.D; no longer Q3.G, R3.1, R4.2
- net N$36: now also D4.A; no longer Q4.G, R7.2
- net N$37: now also D5.C, Q3.D; no longer D5.A, R8.1
- net N$40: now also D5.A, R9.1; no longer Q1.B, R29.2, R30.2, R31.2, R32.2, R33.2, R34.2, R35.2, R36.2
- net N$41: now also D6.C, Q4.D; no longer Q5.G, R10.2, R9.1
- net N$42: now also R12.1; no longer R11.1
- net N$44: now also D7.C, Q5.D; no longer Q6.G, R12.1, R13.2
- net N$45: now also R15.1; no longer R14.1
- net N$46: now also D8.C, Q6.D; no longer D2.A, Q1.E, R37.1
- net N$47: now also D8.A, R19.1; no longer Q7.G, R15.1, R16.2
- net N$48: now also D9.C, Q7.D; no longer D8.A, R17.1
- net N$50: now also D9.A, R22.1; no longer Q8.G, R18.1, R19.2
- net N$51: now also D10.C, Q8.D; no longer D9.A, R20.1
- net N$53: now also D10.A, R25.1; no longer Q9.G, R21.1, R22.2
- net N$56: now also D2.A, R28.1; no longer Q10.G, R24.1, R25.2
Other:
- note added: "Bottom Side"
- note added: "Single Status LED"
- note added: "The value for the top resistor in the voltage dividers above are dependent on the input impedence of the ESC modules. Assuming that they are "high" impedence would heavily effect the value of the voltage divider. If the ESC is high impedence we can short the top resistor. If the ESC are "low" impedence, then the voltage dividers will behave."
- note added: "Top Side"
- note removed: "Bottom"
- note removed: "Top"
- note removed: "Worthy of more consideration"
- note removed: "failed more consideration"
- note removed: "worthy of re-evaluation"
- moved on the sheet: D10, D3, D4, D5, D6, D7, D8, D9, Q3, Q4, Q5, Q6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

Commit message: ESC board updates
Parts:
- removed THRUSTER_PWM_1: 1, pinhead:PINHD-1X3
- removed THRUSTER_PWM_2, THRUSTER_PWM_3, THRUSTER_PWM_4, THRUSTER_PWM_5, THRUSTER_PWM_6, THRUSTER_PWM_7, THRUSTER_PWM_8: (no value), pinhead:PINHD-1X3
- added U$1, U$2, U$3, U$4, U$5, U$6, U$7, U$8: MALE1PINHEADER, Male_Header_1Pin:MALE1PINHEADER
Connections:
- net GND: no longer THRUSTER_PWM_1.3, THRUSTER_PWM_2.3, THRUSTER_PWM_3.3, THRUSTER_PWM_4.3, THRUSTER_PWM_5.3, THRUSTER_PWM_6.3, THRUSTER_PWM_7.3, THRUSTER_PWM_8.3
- net PWM_1: now also U$1.PWM; no longer THRUSTER_PWM_1.1
- net PWM_2: now also U$2.PWM; no longer THRUSTER_PWM_2.1
- net PWM_3: now also U$3.PWM; no longer THRUSTER_PWM_3.1
- net PWM_4: now also U$4.PWM; no longer THRUSTER_PWM_4.1
- net PWM_5: now also U$5.PWM; no longer THRUSTER_PWM_5.1
- net PWM_6: now also U$6.PWM; no longer THRUSTER_PWM_6.1
- net PWM_7: now also U$7.PWM; no longer THRUSTER_PWM_7.1
- net PWM_8: now also U$8.PWM; no longer THRUSTER_PWM_8.1
Other:
- note removed: "Single Status Indicator"
