File: Titan Boards/Actuator/MK1-2/Actuator-MKI-2.brd (EAGLE design)
At the start: 101.6 x 101.6 mm, 61 parts, among them U1 DRV8816PWPR

Commit message: Tempest Actuator MK1-2 Updates
Parts:
- removed D2, D6: (no value), diode:SMB
- removed Q1, Q11, Q15, Q16: (no value), SparkFun-DiscreteSemi:SOT23-3
- removed U$2, U$3: ERZ-VF2M270ERZ-VF2M270, ERZ-VF2M270:RESM8060X320N
- added Q19, Q20: (no value), SparkFun-DiscreteSemi:SOT23-3
- added R1: 5.1k, resistor:R0603
- added R18, R19, R21, R22, R24, R25, R27, R6, R7, R8: 10K, resistor:R0603
- added R2: 7.8k, resistor:R0603
- added R5: 33k, resistor:R0603
- R3: value 10k -> 10K
- R4: value 1 -> 0.5
- moved R3 49.1 mm to (94.9, 65.3), turned to 90 degrees
- moved C16 13.5 mm to (59.3, 52.3), turned to 0 degrees
- moved C19 10.5 mm to (53.7, 38.3), turned to 180 degrees
- moved Q2 5.67 mm to (40.3, 48.4)
- moved Q3 5.67 mm to (35.8, 48.5)
- moved Q12 4.85 mm to (46.7, 42.2)
- moved Q17 4.82 mm to (46.7, 37.9)
- moved D8 4.76 mm to (40.6, 37.5)
- moved D9 4.76 mm to (40.5, 41.7)
- moved C17 2.48 mm to (55.2, 43.8), turned to 0 degrees
- moved C4 2.26 mm to (72.1, 48.3)
- moved C20 2.10 mm to (72.1, 21.5)
- moved R4 2.09 mm to (51.7, 45.7)
- moved C18 0.54 mm to (59.6, 49.4)
Connections:
- removed net COIL_5_GATE: Q11.1, Q15.1, U$9.P$16
- removed net COIL_S_GATE: Q1.1, Q16.1, U$9.P$17
- new net N$3: R2.1, U$6.P$3
- new net N$5: Q19.1, R1.1
- new net N$6: Q19.2, Q20.1, R5.1
- new net N$7: Q20.3, R2.2
- net +24V: no longer D2.C, D6.C
- net +3V3: now also U1.2, U1.5, U1.6; no longer CHARGING.A
- net +5V: no longer R3.2, U1.2, U1.5, U1.6
- net AGND: now also Q19.3, R18.2, R19.2, R21.2, R22.2, R24.2, R25.2, R27.2, R3.2, R6.2, R7.2, R8.2; no longer Q1.2, Q11.2, Q15.2, Q16.2, R3.1, U$2.1, U$3.1
- net ARM_TORPEDO: now also CHARGING.A, R1.2, R27.1, U$9.P$18; no longer U$6.P$3, U$9.P$9
- net COIL_1_GATE: now also R6.1, U$9.P$4; no longer U$9.P$12
- net COIL_2_GATE: now also R24.1, U$9.P$14; no longer U$9.P$13
- net COIL_3_GATE: now also R7.1, U$9.P$5; no longer U$9.P$14
- net COIL_4_GATE: now also R25.1
- net COIL_5: no longer D6.A, Q11.3, Q15.3, U$3.2
- net COIL_S: no longer D2.A, Q1.3, Q16.3, U$2.2
- net DROPPER1_GATE: now also R21.1, U$9.P$3; no longer U$9.P$2
- net DROPPER2_GATE: now also R22.1, U$9.P$13; no longer U$9.P$3
- net PWM_DRIVER1: now also R3.1, U$9.P$9; no longer U$9.P$5
- net PWM_DRIVER2: now also R8.1, U$9.P$19; no longer U$9.P$6
- net SCL: now also U$9.P$17; no longer U$9.P$7
- net SDA: now also U$9.P$7; no longer U$9.P$8
- net TORPEDO1_GATE: now also R18.1, U$9.P$2; no longer U$9.P$18
- net TORPEDO2_GATE: now also R19.1, U$9.P$12; no longer U$9.P$19
- net V+: now also Q20.2, R5.2
Routing:
- net ARM_TORPEDO: track 93.0 -> 188.4 mm, vias 1 -> 7
- net COIL_5_GATE: track 82.9 -> 0.00 mm, vias 2 -> 0
- net COIL_S_GATE: track 80.5 -> 0.00 mm, vias 2 -> 0
- net +3V3: track 193.3 -> 113.4 mm
- net +24V: track 167.2 -> 88.8 mm
- net COIL_5: track 55.4 -> 0.00 mm
- net PWM_DRIVER1: track 29.2 -> 70.0 mm
- net COIL_S: track 38.7 -> 0.00 mm, vias 1 -> 0
- net PWM_DRIVER2: track 28.9 -> 55.2 mm
- net AGND: track 38.6 -> 62.3 mm, vias 21 -> 17
- net N$2: track 18.5 -> 0.00 mm
- net SDA: track 68.0 -> 51.7 mm
- net +5V: track 80.7 -> 65.5 mm, vias 3 -> 2
- net N$6: track 0.00 -> 13.0 mm
- net TORPEDO1_GATE: track 62.4 -> 75.0 mm
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- added copper zone on layer 16, net +12V
- added copper zone on layer 1, net +24V
- added copper zone on layer 1, net N$2
- added copper zone on layer 1, net N$45
- added copper zone on layer 1, net N$48
- added copper zone on layer 1, net N$49
- added copper zone on layer 1, net V+

Commit message: Actuator MK1-2 Updates
Parts:
- removed ARMED: (no value), led:CHIPLED_0603
- added POWER_IN: (no value), led:CHIPLED_0603
- moved R20 23.8 mm to (18.8, 10.5), turned to 0 degrees
- moved Q18 2.49 mm to (23.2, 65.2)
- moved Q6 2.49 mm to (23.2, 56.9)
Connections:
- removed net COIL_5: TORPEDO_CONNECTOR.3
- removed net COIL_S: TORPEDO_CONNECTOR.4
- new net MOTOR_EN: U$9.P$16, U1.2, U1.6
- new net V_DIV: U$9.P$8
- net +24V: no longer R20.2
- net +3V3: no longer U1.2, U1.6
- net AGND: now also POWER_IN.C; no longer ARMED.C
- net N$10: now also POWER_IN.A; no longer ARMED.A
- net V+: now also R20.2
Routing:
- net MOTOR_EN: track 0.00 -> 48.6 mm, vias 0 -> 3
- net +24V: track 88.8 -> 97.4 mm, vias 2 -> 4
- net AGND: track 62.3 -> 66.7 mm
- net V+: track 0.00 -> 3.78 mm
- net N$35: track 10.7 -> 13.3 mm
- net N$33: track 15.4 -> 17.7 mm
- net +3V3: track 113.4 -> 115.2 mm
- net N$10: track 2.31 -> 3.66 mm
- net TORPEDO2: track 26.9 -> 26.2 mm
- net TORPEDO1: track 10.7 -> 9.93 mm
- net ARM_TORPEDO: vias 7 -> 5
- added copper zone on layer 1, net MOTOR_EN

Commit message: Actuator Mk1-2 Updates
Parts:
- added R10: 1K, resistor:R0603
- added R11: 150, resistor:R0603
- added R13: 10K, resistor:R0603
- moved R7 13.3 mm to (60.6, 74.2)
- moved R18 13.2 mm to (77.6, 71.2)
- moved R21 13.2 mm to (69.4, 71.2)
- moved R22 13.2 mm to (66.7, 71.2)
- moved R24 13.2 mm to (72.1, 71.2)
- moved R25 13.2 mm to (74.9, 71.2)
- moved R3 13.2 mm to (83.1, 71.2)
- moved R6 13.2 mm to (63.9, 71.2)
- moved R27 13.2 mm to (80.3, 71.2)
- moved R8 13.2 mm to (85.8, 71.2)
- moved R19 11.5 mm to (67.4, 75.3)
Connections:
- net +24V: now also R10.1
- net AGND: now also R11.2, R13.2
- net MOTOR_EN: now also R13.1
- net V_DIV: now also R10.2, R11.1
Routing:
- net V_DIV: track 0.00 -> 37.9 mm, vias 0 -> 1
- net ARM_TORPEDO: track 188.4 -> 174.4 mm, vias 5 -> 4
- net PWM_DRIVER2: track 55.2 -> 46.5 mm
- net PWM_DRIVER1: track 70.1 -> 63.3 mm
- net TORPEDO1_GATE: track 75.1 -> 68.7 mm
- net COIL_4_GATE: track 75.1 -> 69.6 mm
- net DROPPER2_GATE: track 60.1 -> 56.0 mm, vias 2 -> 1
- net DROPPER1_GATE: track 73.6 -> 69.8 mm, vias 2 -> 1
- net MOTOR_EN: track 48.6 -> 46.1 mm
- net COIL_2_GATE: track 77.5 -> 75.3 mm
- net AGND: track 66.7 -> 65.0 mm
- net COIL_3_GATE: track 64.9 -> 63.7 mm
- net COIL_1_GATE: track 72.9 -> 72.3 mm, vias 3 -> 2
- net TORPEDO2_GATE: track 61.2 -> 61.5 mm, vias 2 -> 1
Other:
- board text added: "The Underwater Robotics Team"
- board text removed: "The Underwater Robotics Team Center for Automotive Research"
