File: Titan Boards/Actuator/MK1-3/Actuator-MKI-3.sch (EAGLE design)
At the start: 57 parts, among them Q12 MOSFET-NCH-AO3404A, Q17 MOSFET-NCH-AO3404A, Q18 FDD4141TO252, Q2 MOSFET-NCH-AO3404A, Q3 MOSFET-NCH-AO3404A, Q6 FDD4141TO252, U1 DRV8816PWPR, U2 MBRB2060CTT4G, U3 MBRB2060CTT4G, U4 MBRB2060CTT4G, U5 MBRB2060CTT4G, U6 MBRB2060CTT4G, U7 MBRB2060CTT4G

Commit message: Actuator MK1-3 updates
Parts:
- R10: value 1K -> 10K
- R11: value 150 -> 1.5K
Connections:
- new net VPROPI: U$9.P$6, U1.VPROPI
Other:
- note added: "3.5 mm screw terminal Either two 2-pos or one 4-pos"
Changed lines of the file:
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@@
 <part name="P+2" library="supply1" library_urn="urn:adsk.eagle:library:371" deviceset="V+" device=""/>
 <part name="P+11" library="supply1" library_urn="urn:adsk.eagle:library:371" deviceset="+24V" device=""/>
-<part name="R10" library="resistor" library_urn="urn:adsk.eagle:library:348" deviceset="R-US_" device="R0603" package3d_urn="urn:adsk.eagle:package:23555/2" value="1K"/>
-<part name="R11" library="resistor" library_urn="urn:adsk.eagle:library:348" deviceset="R-US_" device="R0603" package3d_urn="urn:adsk.eagle:package:23555/2" value="150"/>
+<part name="R10" library="resistor" library_urn="urn:adsk.eagle:library:348" deviceset="R-US_" device="R0603" package3d_urn="urn:adsk.eagle:package:23555/2" value="10K"/>
+<part name="R11" library="resistor" library_urn="urn:adsk.eagle:library:348" deviceset="R-US_" device="R0603" package3d_urn="urn:adsk.eagle:package:23555/2" value="1.5K"/>
 <part name="AGND1" library="supply1" library_urn="urn:adsk.eagle:library:371" deviceset="AGND" device=""/>
 <part name="R13" library="resistor" library_urn="urn:adsk.eagle:library:348" deviceset="R-US_" device="R0603" package3d_urn="urn:adsk.eagle:package:23555/2" value="10K"/>
@@
 <text x="157.48" y="195.58" size="2.54" layer="91">Voltage Divider</text>
 <text x="40.64" y="193.04" size="1.778" layer="91">High rated DPAK2 footprint NMOS</text>
+<text x="177.8" y="33.02" size="1.778" layer="91">3.5 mm screw terminal
+Either two 2-pos or
+one 4-pos</text>
 </plain>
 <instances>
@@
 <net name="SDA" class="0">
 <segment>
-<wire x1="264.16" y1="144.78" x2="264.16" y2="165.1" width="0.1524" layer="91"/>
-<label x="264.16" y="165.1" size="1.778" layer="95" rot="R90" xref="yes"/>
+<wire x1="259.08" y1="144.78" x2="259.08" y2="165.1" width="0.1524" layer="91"/>
+<label x="259.08" y="165.1" size="1.778" layer="95" rot="R90" xref="yes"/>
 <pinref part="U$9" gate="G$1" pin="P$7"/>
-<wire x1="287.02" y1="144.78" x2="264.16" y2="144.78" width="0.1524" layer="91"/>
+<wire x1="287.02" y1="144.78" x2="259.08" y2="144.78" width="0.1524" layer="91"/>
 </segment>
 <segment>
@@
 </segment>
 <segment>
-<wire x1="254" y1="139.7" x2="254" y2="165.1" width="0.1524" layer="91"/>
-<label x="254" y="165.1" size="1.778" layer="95" rot="R90" xref="yes"/>
+<wire x1="248.92" y1="139.7" x2="248.92" y2="165.1" width="0.1524" layer="91"/>
+<label x="248.92" y="165.1" size="1.778" layer="95" rot="R90" xref="yes"/>
 <pinref part="U$9" gate="G$1" pin="P$9"/>
-<wire x1="254" y1="139.7" x2="263.398" y2="139.7" width="0.1524" layer="91"/>
+<wire x1="248.92" y1="139.7" x2="258.318" y2="139.7" width="0.1524" layer="91"/>
 <pinref part="R3" gate="G$1" pin="1"/>
-<wire x1="264.16" y1="139.7" x2="287.02" y2="139.7" width="0.1524" layer="91"/>
-<wire x1="263.398" y1="137.16" x2="263.398" y2="139.7" width="0.1524" layer="91"/>
-<wire x1="263.398" y1="139.7" x2="264.16" y2="139.7" width="0.1524" layer="91"/>
-<junction x="264.16" y="139.7"/>
+<wire x1="259.08" y1="139.7" x2="287.02" y2="139.7" width="0.1524" layer="91"/>
+<wire x1="263.398" y1="137.16" x2="258.318" y2="139.7" width="0.1524" layer="91"/>
+<wire x1="258.318" y1="139.7" x2="259.08" y2="139.7" width="0.1524" layer="91"/>
+<junction x="259.08" y="139.7"/>
 </segment>
 </net>
@@
 <segment>
 <pinref part="U$9" gate="G$1" pin="P$8"/>
-<wire x1="287.02" y1="142.24" x2="259.08" y2="142.24" width="0.1524" layer="91"/>
-<wire x1="259.08" y1="142.24" x2="259.08" y2="165.1" width="0.1524" layer="91"/>
-<label x="259.08" y="165.1" size="1.778" layer="95" rot="R90" xref="yes"/>
+<wire x1="287.02" y1="142.24" x2="254" y2="142.24" width="0.1524" layer="91"/>
+<wire x1="254" y1="142.24" x2="254" y2="165.1" width="0.1524" layer="91"/>
+<label x="254" y="165.1" size="1.778" layer="95" rot="R90" xref="yes"/>
 </segment>
 <segment>
@@
 </segment>
 </net>
+<net name="VPROPI" class="0">
+<segment>
+<pinref part="U$9" gate="G$1" pin="P$6"/>
+<wire x1="287.02" y1="147.32" x2="264.16" y2="147.32" width="0.1524" layer="91"/>
+<wire x1="264.16" y1="147.32" x2="264.16" y2="165.1" width="0.1524" layer="91"/>
+<label x="264.16" y="165.1" size="1.778" layer="95" rot="R90" xref="yes"/>
+</segment>
+<segment>
+<pinref part="U1" gate="A" pin="VPROPI"/>
+<wire x1="313.182" y1="236.22" x2="317.5" y2="236.22" width="0.1524" layer="91"/>
+<wire x1="317.5" y1="236.22" x2="317.5" y2="241.3" width="0.1524" layer="91"/>
+<label x="317.5" y="241.3" size="1.778" layer="95" xref="yes"/>
+</segment>
+</net>

Commit message: Actuator MKIII updates'
Parts:
- removed C20, C4: UVK1E223MRD, UVK1E223MRD:UVK1E223MRD
- added U$1: 31059104, 31059104:31059104
Connections:
- net +24V: now also U$1.P$1, U$1.P$2; no longer C20.1, C4.1
- net AGND: now also U$1.P$3, U$1.P$4; no longer C20.2, C4.2
Changed lines of the file:
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@@
 <part name="C17" library="rcl" library_urn="urn:adsk.eagle:library:334" deviceset="C-EU" device="C0603" package3d_urn="urn:adsk.eagle:package:23616/2" value="0.1uF"/>
 <part name="C19" library="25TZV100M6_3X8" deviceset="25TZV100M6.3X8" device=""/>
-<part name="C4" library="UVK1E223MRD" deviceset="UVK1E223MRD" device=""/>
-<part name="C20" library="UVK1E223MRD" deviceset="UVK1E223MRD" device=""/>
 <part name="AGND44" library="supply1" library_urn="urn:adsk.eagle:library:371" deviceset="AGND" device=""/>
 <part name="U$9" library="JTAG-SMD" deviceset="JTAG-SMD" device=""/>
@@
 <part name="U6" library="DPAK2" deviceset="MBRB2060CTT4G" device=""/>
 <part name="U7" library="DPAK2" deviceset="MBRB2060CTT4G" device=""/>
+<part name="U$1" library="31059104" deviceset="31059104" device=""/>
+<part name="P+3" library="supply1" library_urn="urn:adsk.eagle:library:371" deviceset="+24V" device=""/>
+<part name="AGND7" library="supply1" library_urn="urn:adsk.eagle:library:371" deviceset="AGND" device=""/>
 </parts>
 <sheets>
@@
 <attribute name="NAME" x="347.7768" y="230.6574" size="1.27" layer="95" ratio="10" rot="SR270"/>
 </instance>
-<instance part="C4" gate="A" x="302.768" y="82.042" smashed="yes" rot="R270">
-<attribute name="VALUE" x="299.7708" y="81.6102" size="0.762" layer="96" ratio="10" rot="SR270"/>
-<attribute name="NAME" x="301.2948" y="77.2414" size="1.524" layer="95" ratio="10" rot="SR270"/>
-</instance>
-<instance part="C20" gate="A" x="297.18" y="82.042" smashed="yes" rot="R270">
-<attribute name="VALUE" x="293.6748" y="81.1022" size="0.762" layer="96" ratio="10" rot="SR270"/>
-<attribute name="NAME" x="296.3672" y="73.3806" size="1.524" layer="95" ratio="10" rot="SR90"/>
-</instance>
 <instance part="AGND44" gate="VR1" x="299.72" y="119.38" smashed="yes">
 <attribute name="VALUE" x="299.72" y="116.84" size="1.778" layer="96" rot="R180"/>
@@
 <instance part="U6" gate="A" x="228.6" y="81.28" smashed="yes" rot="MR180"/>
 <instance part="U7" gate="A" x="220.98" y="76.2" smashed="yes" rot="MR180"/>
+<instance part="U$1" gate="G$1" x="116.84" y="43.18" smashed="yes"/>
+<instance part="P+3" gate="1" x="129.54" y="55.88" smashed="yes">
+<attribute name="VALUE" x="127" y="50.8" size="1.778" layer="96" rot="R90"/>
+</instance>
+<instance part="AGND7" gate="VR1" x="129.54" y="30.48" smashed="yes">
+<attribute name="VALUE" x="139.7" y="30.48" size="1.778" layer="96" rot="MR0"/>
+</instance>
 </instances>
 <busses>
@@
 <wire x1="299.72" y1="71.12" x2="299.72" y2="68.58" width="0.1524" layer="91"/>
 <wire x1="309.88" y1="76.2" x2="309.88" y2="71.12" width="0.1524" layer="91"/>
-<wire x1="309.88" y1="71.12" x2="302.768" y2="71.12" width="0.1524" layer="91"/>
+<wire x1="309.88" y1="71.12" x2="299.72" y2="71.12" width="0.1524" layer="91"/>
 <junction x="299.72" y="71.12"/>
 <pinref part="C5" gate="G$1" pin="2"/>
-<wire x1="302.768" y1="71.12" x2="299.72" y2="71.12" width="0.1524" layer="91"/>
 <wire x1="279.4" y1="73.66" x2="279.4" y2="71.12" width="0.1524" layer="91"/>
-<wire x1="279.4" y1="71.12" x2="297.18" y2="71.12" width="0.1524" layer="91"/>
+<wire x1="279.4" y1="71.12" x2="299.72" y2="71.12" width="0.1524" layer="91"/>
 <pinref part="POWER_IN" gate="G$1" pin="C"/>
-<wire x1="297.18" y1="71.12" x2="299.72" y2="71.12" width="0.1524" layer="91"/>
 <wire x1="312.42" y1="71.12" x2="309.88" y2="71.12" width="0.1524" layer="91"/>
 <junction x="309.88" y="71.12"/>
-<pinref part="C20" gate="A" pin="2"/>
-<wire x1="297.18" y1="74.422" x2="297.18" y2="71.12" width="0.1524" layer="91"/>
-<junction x="297.18" y="71.12"/>
-<pinref part="C4" gate="A" pin="2"/>
-<wire x1="302.768" y1="74.422" x2="302.768" y2="71.12" width="0.1524" layer="91"/>
-<junction x="302.768" y="71.12"/>
 </segment>
 <segment>
@@
 <wire x1="55.88" y1="43.18" x2="55.88" y2="35.56" width="0.1524" layer="91"/>
 </segment>
+<segment>
+<pinref part="AGND7" gate="VR1" pin="AGND"/>
+<pinref part="U$1" gate="G$1" pin="P$4"/>
+<wire x1="129.54" y1="33.02" x2="129.54" y2="35.56" width="0.1524" layer="91"/>
+<wire x1="129.54" y1="35.56" x2="124.46" y2="35.56" width="0.1524" layer="91"/>
+<pinref part="U$1" gate="G$1" pin="P$3"/>
+<wire x1="124.46" y1="40.64" x2="129.54" y2="40.64" width="0.1524" layer="91"/>
+<wire x1="129.54" y1="40.64" x2="129.54" y2="35.56" width="0.1524" layer="91"/>
+<junction x="129.54" y="35.56"/>
+</segment>
 </net>
 <net name="SDA" class="0">
@@
 </segment>
 <segment>
-<wire x1="294.64" y1="86.36" x2="297.18" y2="86.36" width="0.1524" layer="91"/>
 <pinref part="D10" gate="G$1" pin="C"/>
-<wire x1="297.18" y1="86.36" x2="302.768" y2="86.36" width="0.1524" layer="91"/>
-<wire x1="302.768" y1="86.36" x2="309.88" y2="86.36" width="0.1524" layer="91"/>
+<wire x1="294.64" y1="86.36" x2="309.88" y2="86.36" width="0.1524" layer="91"/>
 <wire x1="309.88" y1="86.36" x2="309.88" y2="81.28" width="0.1524" layer="91"/>
 <pinref part="P+8" gate="1" pin="+24V"/>
@@
 <junction x="309.88" y="86.36"/>
 <pinref part="120" gate="G$1" pin="2"/>
-<pinref part="C20" gate="A" pin="1"/>
-<wire x1="297.18" y1="82.042" x2="297.18" y2="86.36" width="0.1524" layer="91"/>
-<junction x="297.18" y="86.36"/>
-<pinref part="C4" gate="A" pin="1"/>
-<wire x1="302.768" y1="82.042" x2="302.768" y2="86.36" width="0.1524" layer="91"/>
-<junction x="302.768" y="86.36"/>
 </segment>
 <segment>
@@
 <wire x1="179.578" y1="187.96" x2="182.88" y2="187.96" width="0.1524" layer="91"/>
 </segment>
+<segment>
+<pinref part="P+3" gate="1" pin="+24V"/>
+<pinref part="U$1" gate="G$1" pin="P$1"/>
+<wire x1="129.54" y1="53.34" x2="129.54" y2="50.8" width="0.1524" layer="91"/>
+<wire x1="129.54" y1="50.8" x2="124.46" y2="50.8" width="0.1524" layer="91"/>
+<pinref part="U$1" gate="G$1" pin="P$2"/>
+<wire x1="129.54" y1="50.8" x2="129.54" y2="45.72" width="0.1524" layer="91"/>
+<wire x1="129.54" y1="45.72" x2="124.46" y2="45.72" width="0.1524" layer="91"/>
+<junction x="129.54" y="50.8"/>
+</segment>
 </net>

Commit message: Actuator MK3 for Review
Parts:
- renumbered U$9 to U$2
Connections:
- net ARM_TORPEDO: now also U$2.P$6; no longer U$2.P$18
- net COIL_1_GATE: now also R24.1, U$2.P$14; no longer R6.1, U$2.P$4
- net COIL_2_GATE: now also R6.1, U$2.P$4; no longer R24.1, U$2.P$14
- net COIL_3_GATE: now also R25.1, U$2.P$15; no longer R7.1, U$2.P$5
- net COIL_4_GATE: now also R7.1, U$2.P$5; no longer R25.1, U$2.P$15
- net SCL: now also U$2.P$7; no longer U$2.P$17
- net SDA: now also U$2.P$17; no longer U$2.P$7
- net VPROPI: now also U$2.P$18; no longer U$2.P$6
Other:
- note added: "3.5 mm screw terminal pitch"
- note added: "Additional Standard Components: · Resistors · Capacitors · Polarized Capacitors · LEDs · Suppressor Diodes"
- note added: "Administrative Notes: Board Name: Tempest Acuator Schematic Creation: 04/2022 Schematic Designer(s): Dylan Trainor Electrical Lead: Phillip Barker"
- note added: "COIL signals must be placed on sequential pin numbers for firmware."
- note added: "Capacitor Terminal Block"
- note removed: "3.5 mm screw terminal Either two 2-pos or one 4-pos"
- note removed: "Additional Standard Components: · Resistors · Capacitors · Polarized Capacitors · LEDs · Suppressor Diodes · Switch"
- note removed: "Administrative Notes: Board Name: Titan Acuator Schematic Creation: 09/2020 Schematic Designer(s): Dylan Trainor, Tanner Lapp Electrical Lead: Phillip Barker"
- moved on the sheet: R27, R3

Commit message: Tempest Actuator Board Review Revisions
Parts:
- removed U6, U7: MBRB2060CTT4G, DPAK2:MBRB2060CTT4G
- added Q1, Q4: MOSFET-NCH-AO3404A, SparkFun-DiscreteSemi:MOSFET-NCH-AO3404A
Connections:
- removed net EXTRA5: BACKPLANE_CONN.3
- removed net EXTRA6: BACKPLANE_CONN.1
- net +3V3: now also BACKPLANE_CONN.1; no longer BACKPLANE_CONN.2
- net AGND: now also Q1.D; no longer U7.D
- net N$5: now also Q1.G; no longer U7.G
- net N$6: now also Q1.S, Q4.G; no longer U6.G, U7.S
- net N$7: now also Q4.D; no longer U6.D
- net PWM_OUT2: now also CLAW_CONN.2; no longer CLAW_CONN.3
- net TORPEDO2: now also TORPEDO_CONN.4; no longer TORPEDO_CONN.2
- net V+: now also Q4.S; no longer U6.S
Changed lines of the file:
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@@
 <part name="U4" library="DPAK2" deviceset="MBRB2060CTT4G" device=""/>
 <part name="U5" library="DPAK2" deviceset="MBRB2060CTT4G" device=""/>
-<part name="U6" library="DPAK2" deviceset="MBRB2060CTT4G" device=""/>
-<part name="U7" library="DPAK2" deviceset="MBRB2060CTT4G" device=""/>
 <part name="U$1" library="31059104" deviceset="31059104" device=""/>
 <part name="P+3" library="supply1" library_urn="urn:adsk.eagle:library:371" deviceset="+24V" device=""/>
 <part name="AGND7" library="supply1" library_urn="urn:adsk.eagle:library:371" deviceset="AGND" device=""/>
 <part name="U$2" library="JTAG-SMD" deviceset="JTAG-SMD" device=""/>
+<part name="Q1" library="SparkFun-DiscreteSemi" deviceset="MOSFET-NCH" device="-AO3404A" value=""/>
+<part name="Q4" library="SparkFun-DiscreteSemi" deviceset="MOSFET-NCH" device="-AO3404A" value=""/>
 </parts>
 <sheets>
@@
 <attribute name="VALUE" x="66.04" y="53.34" size="1.778" layer="96" rot="R90"/>
 </instance>
-<instance part="+3V1" gate="G$1" x="60.96" y="58.42" smashed="yes">
-<attribute name="VALUE" x="58.42" y="53.34" size="1.778" layer="96" rot="R90"/>
+<instance part="+3V1" gate="G$1" x="30.48" y="58.42" smashed="yes">
+<attribute name="VALUE" x="27.94" y="53.34" size="1.778" layer="96" rot="R90"/>
 </instance>
 <instance part="AGND2" gate="VR1" x="55.88" y="33.02" smashed="yes">
@@
 <instance part="U4" gate="A" x="83.82" y="177.8" smashed="yes"/>
 <instance part="U5" gate="A" x="109.22" y="177.8" smashed="yes"/>
-<instance part="U6" gate="A" x="228.6" y="81.28" smashed="yes" rot="MR180"/>
-<instance part="U7" gate="A" x="220.98" y="76.2" smashed="yes" rot="MR180"/>
 <instance part="U$1" gate="G$1" x="116.84" y="43.18" smashed="yes"/>
 <instance part="P+3" gate="1" x="129.54" y="55.88" smashed="yes">
@@
 </instance>
 <instance part="U$2" gate="G$1" x="309.88" y="139.7" smashed="yes"/>
+<instance part="Q1" gate="NMOS" x="218.44" y="76.2" smashed="yes" rot="MR180">
+<attribute name="NAME" x="223.52" y="76.2" size="1.778" layer="95" font="vector" rot="MR180"/>
+<attribute name="VALUE" x="223.52" y="78.74" size="1.778" layer="96" font="vector" rot="MR180"/>
+</instance>
+<instance part="Q4" gate="NMOS" x="226.06" y="81.28" smashed="yes" rot="MR180">
+<attribute name="NAME" x="231.14" y="81.28" size="1.778" layer="95" font="vector" rot="MR180"/>
+<attribute name="VALUE" x="231.14" y="83.82" size="1.778" layer="96" font="vector" rot="MR180"/>
+</instance>
 </instances>
 <busses>
@@
 </segment>
 <segment>
-<pinref part="BACKPLANE_CONN" gate="G$1" pin="2"/>
 <pinref part="+3V1" gate="G$1" pin="+3V3"/>
-<wire x1="53.34" y1="50.8" x2="60.96" y2="50.8" width="0.1524" layer="91"/>
-<wire x1="60.96" y1="50.8" x2="60.96" y2="55.88" width="0.1524" layer="91"/>
+<wire x1="30.48" y1="50.8" x2="30.48" y2="55.88" width="0.1524" layer="91"/>
+<pinref part="BACKPLANE_CONN" gate="G$1" pin="1"/>
+<wire x1="38.1" y1="50.8" x2="30.48" y2="50.8" width="0.1524" layer="91"/>
 </segment>
 </net>
@@
 <wire x1="220.98" y1="71.12" x2="220.98" y2="68.58" width="0.1524" layer="91"/>
 <junction x="220.98" y="68.58"/>
-<pinref part="U7" gate="A" pin="D"/>
+<pinref part="Q1" gate="NMOS" pin="D"/>
 </segment>
 <segment>
@@
 <wire x1="200.66" y1="86.36" x2="200.66" y2="82.042" width="0.1524" layer="91"/>
 <junction x="200.66" y="86.36"/>
-<pinref part="U6" gate="A" pin="S"/>
+<pinref part="Q4" gate="NMOS" pin="S"/>
 <junction x="228.6" y="86.36"/>
 </segment>
@@
 </segment>
 <segment>
-<pinref part="TORPEDO_CONN" gate="G$1" pin="2"/>
-<wire x1="45.72" y1="238.76" x2="63.5" y2="238.76" width="0.1524" layer="91"/>
-<wire x1="63.5" y1="238.76" x2="63.5" y2="231.14" width="0.1524" layer="91"/>
-<label x="63.5" y="231.14" size="1.778" layer="95" rot="R270" xref="yes"/>
+<pinref part="TORPEDO_CONN" gate="G$1" pin="4"/>
+<wire x1="45.72" y1="236.22" x2="60.96" y2="236.22" width="0.1524" layer="91"/>
+<wire x1="60.96" y1="236.22" x2="60.96" y2="231.14" width="0.1524" layer="91"/>
+<label x="60.96" y="231.14" size="1.778" layer="95" rot="R270" xref="yes"/>
 </segment>
 </net>
@@
 </segment>
 <segment>
-<pinref part="CLAW_CONN" gate="G$1" pin="3"/>
-<wire x1="96.52" y1="215.9" x2="88.9" y2="215.9" width="0.1524" layer="91"/>
-<label x="88.9" y="215.9" size="1.778" layer="95" rot="R180" xref="yes"/>
+<pinref part="CLAW_CONN" gate="G$1" pin="2"/>
+<wire x1="111.76" y1="218.44" x2="114.3" y2="218.44" width="0.1524" layer="91"/>
+<wire x1="114.3" y1="218.44" x2="114.3" y2="208.28" width="0.1524" layer="91"/>
+<wire x1="114.3" y1="208.28" x2="88.9" y2="208.28" width="0.1524" layer="91"/>
+<label x="88.9" y="208.28" size="1.778" layer="95" rot="R180" xref="yes"/>
 </segment>
 </net>
@@
 <wire x1="210.82" y1="76.962" x2="213.36" y2="76.962" width="0.1524" layer="91"/>
 <wire x1="213.36" y1="76.962" x2="213.36" y2="78.74" width="0.1524" layer="91"/>
-<pinref part="U7" gate="A" pin="G"/>
 <wire x1="213.36" y1="78.74" x2="214.63" y2="78.74" width="0.1524" layer="91"/>
+<pinref part="Q1" gate="NMOS" pin="G"/>
+<junction x="213.36" y="78.74"/>
 </segment>
 </net>
@@
 <wire x1="210.82" y1="82.042" x2="220.98" y2="82.042" width="0.1524" layer="91"/>
 <wire x1="220.98" y1="82.042" x2="220.98" y2="81.28" width="0.1524" layer="91"/>
-<pinref part="U7" gate="A" pin="S"/>
-<pinref part="U6" gate="A" pin="G"/>
-<wire x1="220.98" y1="83.82" x2="222.25" y2="83.82" width="0.1524" layer="91"/>
+<pinref part="Q1" gate="NMOS" pin="S"/>
+<pinref part="Q4" gate="NMOS" pin="G"/>
 </segment>
 </net>
@@
 <wire x1="228.6" y1="66.04" x2="251.46" y2="66.04" width="0.1524" layer="91"/>
 <wire x1="251.46" y1="66.04" x2="251.46" y2="66.802" width="0.1524" layer="91"/>
-<pinref part="U6" gate="A" pin="D"/>
+<pinref part="Q4" gate="NMOS" pin="D"/>
 </segment>
 </net>
@@
 </segment>
 </net>
-<net name="EXTRA5" class="0">
-<segment>
-<pinref part="BACKPLANE_CONN" gate="G$1" pin="3"/>
-<wire x1="38.1" y1="48.26" x2="25.4" y2="48.26" width="0.1524" layer="91"/>
-<label x="25.4" y="48.26" size="1.778" layer="95" rot="R270" xref="yes"/>
-</segment>
-</net>
 <net name="+5V" class="0">
 <segment>
@@
 </segment>
 </net>
-<net name="EXTRA6" class="0">
-<segment>
-<pinref part="BACKPLANE_CONN" gate="G$1" pin="1"/>
-<wire x1="38.1" y1="50.8" x2="20.32" y2="50.8" width="0.1524" layer="91"/>
-<label x="20.32" y="50.8" size="1.778" layer="95" rot="R270" xref="yes"/>
-</segment>
-</net>
